File: 3350-dual-vcf/3350-dual-vcf.sch (KiCad schematic (older format))
At the start: 5 parts

Commit message: More stuff on 3350 vcf
Parts:
- removed C? (x2): C, symbol Device:C
- removed U? (x3): LM13700, symbol Amplifier_Operational:LM13700
- added C? (x4): 22nF, symbol Device:C
- added J? (x4): AUDIO_IN, symbol EurorackHardware:EurorackJackMono
- added J? (x4): BP_OUT, symbol EurorackHardware:EurorackJackMono
- added R? (x4): 100k, symbol Device:R
- added R? (x4): 33k, symbol Device:R
- added R? (x4): 10k, symbol Device:R
- added R? (x10): 220R, symbol Device:R
- added R? (x6): 22k, symbol Device:R
- added R? (x2): 150k, symbol Device:R
- added RV? (x4): 100kA, symbol Device:R_POT
- added U? (x2): TL074, symbol Audio_Chips:AS3350
- added U? (x10): TL074, symbol Amplifier_Operational:TL074
Connections:
- net GND: now also C?.2, C?.2, C?.2, C?.2, J?.~ (P3), J?.~ (P3), J?.~ (P3), J?.~ (P3), J?.~ (P3), J?.~ (P3), J?.~ (P3), J?.~ (P3), R?.1, R?.1, R?.1, R?.1, R?.1, R?.1, R?.2, R?.2, R?.2, R?.2, RV?.3, RV?.3, RV?.3, RV?.3, U?.3 (+), U?.3 (+), U?.3 (+), U?.3 (+)
- new net: R?.1, R?.1, R?.2, U?.2 (Vif) (x2)
- new net: C?.1, U?.12 (+), U?.3 (Vlp) (x2)
- new net: R?.1, R?.2, U?.4 (Viv) (x2)
- new net: C?.1, U?.10 (+), U?.5 (+), U?.5 (Vbp) (x2)
- new net: J?.~ (P3), RV?.1 (x4)
- new net: R?.2, RV?.2 (x4)
- new net: R?.1, R?.2, U?.1 (x4)
- new net: R?.1, R?.2, U?.2 (-) (x4)
- new net: R?.2, R?.2, U?.6 (-) (x2)
- new net: R?.1, R?.2, U?.7 (x2)
- new net: R?.1, R?.1, U?.9 (-) (x2)
- new net: J?.~ (P3), R?.2, U?.8 (x2)
- new net: R?.1, R?.1, U?.13 (-) (x2)
- new net: J?.~ (P3), R?.2, U?.14 (x2)
- new net FREQ_CV1: U?.6 (Vcq), U?.6 (Vcq)
- new net Q_CV1: U?.8 (Vcf), U?.8 (Vcf)
- no-connect marks 0 -> 8
