File: serge-gain-cell/serge-gain-cell.sch (KiCad schematic (older format))
At the start: 20 parts, among them J1 Conn_01x08_Male, Q1 2N3904, Q2 2N3906, Q3 2N3904, Q4 2N3906, U1 LF353

Commit message: More updates to gain cell
Parts:
- C1, C2, C3, C4: footprint (none) -> Capacitor_THT:C_Disc_D4.7mm_W2.5mm_P5.00mm
- D1, D2: footprint (none) -> rumblesan-footprints:Diode_THT_P7.62mm_Horizontal
- J1: footprint (none) -> Connector_PinHeader_2.54mm:PinHeader_1x08_P2.54mm_Vertical
- R1, R2, R3, R4, R5, R6, R7: footprint (none) -> rumblesan-footprints:Resistor_THT_L6.3mm_D2.5mm_P10.16mm_Horizontal
- RV1: footprint (none) -> rumblesan-footprints:Potentiometer_THT_Bourns_3306P_Vertical
- U1: footprint (none) -> Package_DIP:DIP-8_W7.62mm_Socket
- renumbered Q2 to Q1, Q4 to Q2, Q1 to Q3, Q3 to Q4
Connections:
- net In: now reaches C1.2, J1.4 (Pin_4), Q1.3 (C), Q3.3 (C), U1.2 (-)
- net FB: now reaches C2.2, J1.6 (Pin_6), Q2.3 (C), Q4.3 (C), U1.6 (-)
- net Out: now reaches C2.1, J1.5 (Pin_5), U1.7
- net CV: now reaches J1.7 (Pin_7), R5.2
Other:
- moved on the sheet: C2, J1, R5, U1B
