File: serge-gain-cell/serge-gain-cell.kicad_pcb (KiCad board)
At the start: 2 copper layers, 0 parts

Commit message: More updates to gain cell
Parts:
- added C1: 47pF, Capacitor_THT:C_Disc_D4.7mm_W2.5mm_P5.00mm, F.Cu at (141.5, 65.5)
- added C2: 5pF, Capacitor_THT:C_Disc_D4.7mm_W2.5mm_P5.00mm, F.Cu at (126.0, 67.5)
- added C3: 10nF, Capacitor_THT:C_Disc_D4.7mm_W2.5mm_P5.00mm, F.Cu at (126.0, 70.0)
- added C4: 10nF, Capacitor_THT:C_Disc_D4.7mm_W2.5mm_P5.00mm, F.Cu at (126.0, 55.0)
- added D1: 1n4148, rumblesan-footprints:Diode_THT_P7.62mm_Horizontal, F.Cu at (153.5, 64.1)
- added D2: 1n4148, rumblesan-footprints:Diode_THT_P7.62mm_Horizontal, F.Cu at (150.0, 64.1)
- added J1: Conn_01x08_Male, Connector_PinHeader_2.54mm:PinHeader_1x08_P2.54mm_Vertical, F.Cu at (126.5, 79.5)
- added Q1: 2N3906, Package_TO_SOT_THT:TO-92_Inline, F.Cu at (151.0, 76.5)
- added Q2: 2N3906, Package_TO_SOT_THT:TO-92_Inline, F.Cu at (157.5, 76.5)
- added Q3: 2N3904, Package_TO_SOT_THT:TO-92_Inline, F.Cu at (150.5, 67.5)
- added Q4: 2N3904, Package_TO_SOT_THT:TO-92_Inline, F.Cu at (157.0, 67.5)
- added R1: 8k2, rumblesan-footprints:Resistor_THT_L6.3mm_D2.5mm_P10.16mm_Horizontal, F.Cu at (146.7, 73.0)
- added R2: 8k2, rumblesan-footprints:Resistor_THT_L6.3mm_D2.5mm_P10.16mm_Horizontal, F.Cu at (136.5, 70.0)
- added R3: 150k, rumblesan-footprints:Resistor_THT_L6.3mm_D2.5mm_P10.16mm_Horizontal, F.Cu at (128.5, 76.0)
- added R4: 150k, rumblesan-footprints:Resistor_THT_L6.3mm_D2.5mm_P10.16mm_Horizontal, F.Cu at (139.2, 55.5)
- added R5: 100R, rumblesan-footprints:Resistor_THT_L6.3mm_D2.5mm_P10.16mm_Horizontal, F.Cu at (145.5, 55.3)
- added R6: 1M5, rumblesan-footprints:Resistor_THT_L6.3mm_D2.5mm_P10.16mm_Horizontal, F.Cu at (162.0, 66.0)
- added R7: 330R, rumblesan-footprints:Resistor_THT_L6.3mm_D2.5mm_P10.16mm_Horizontal, F.Cu at (158.4, 79.8)
- added RV1: 100k, rumblesan-footprints:Potentiometer_THT_Bourns_3306P_Vertical, F.Cu at (160.5, 59.0)
- added U1: LF353, Package_DIP:DIP-8_W7.62mm_Socket, F.Cu at (137.1, 66.6)
Routing:
- net GNDREF: track 0.00 -> 93.1 mm, vias 0 -> 1
- net +12V: track 0.00 -> 63.5 mm
- net -12V: track 0.00 -> 63.5 mm
- net /FB: track 0.00 -> 50.6 mm
- net Net-(D2-Pad2): track 0.00 -> 41.8 mm
- net /In: track 0.00 -> 41.0 mm
- net Net-(D1-Pad1): track 0.00 -> 36.7 mm
- net Net-(Q1-Pad2): track 0.00 -> 29.6 mm
- net /Out: track 0.00 -> 21.3 mm
- net /CV: track 0.00 -> 15.6 mm
- net Net-(C1-Pad1): track 0.00 -> 12.0 mm
- net Net-(R6-Pad1): track 0.00 -> 10.1 mm
- net Net-(Q2-Pad2): track 0.00 -> 9.95 mm
- added copper zone on B.Cu, net GNDREF
- added copper zone on F.Cu, net GNDREF
Other:
- board outline added: 40.5 x 28 mm

Commit message: Updating ordered boards
Other:
- outline, holes or cut-outs redrawn
- rule pad_to_mask_clearance: 0.0508 -> 0
