File: cgs348-vco-output-buffer/cgs348-vco-output-buffer.sch (KiCad schematic (older format))
At the start: 27 parts, among them J1 Wire_24AWG_Stranded, J2 Wire_24AWG_Stranded, J3 Wire_24AWG_Stranded, J4 Wire_24AWG_Stranded, J5 Wire_24AWG_Stranded, J6 Wire_24AWG_Stranded, J7 Wire_24AWG_Stranded, J8 Wire_24AWG_Stranded, J9 Power, U1 TL074

Commit message: Updating ordered boards
Parts:
- removed H3: Logo_Ammonite-simple, rumblesan-footprints:Logo_Ammonite-simple_10.4mmx12.0mm, symbol Board_Hardware:Logo_Ammonite-simple
- added R10, R11, R12, R13, R14, R15, R16, R9: 47k, rumblesan-footprints:Resistor_THT_L6.3mm_D2.5mm_P10.16mm_Horizontal, symbol Device:R
Connections:
- net GND: now also R13.2, R14.2, R15.2, R16.2
- net at J1.1: now also R9.1; no longer U1.3 (+)
- net at J2.1: now also R10.1; no longer U1.5 (+)
- net at J3.1: now also R11.1; no longer U1.10 (+)
- net at J4.1: now also R12.1; no longer U1.12 (+)
- new net: R13.1, R9.2, U1.3 (+)
- new net: R10.2, R14.1, U1.5 (+)
- new net: R11.2, R15.1, U1.10 (+)
- new net: R12.2, R16.1, U1.12 (+)
Other:
- moved on the sheet: J1, J2, J3, J4, J5, J6, J7, J8, R1, R2, R3, R4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
