File: cgs348-vco-output-buffer/cgs348-vco-output-buffer.kicad_sch (KiCad schematic)
At the start: 28 parts, among them J1 Wire_24AWG_Stranded, J2 Wire_24AWG_Stranded, J3 Wire_24AWG_Stranded, J4 Wire_24AWG_Stranded, J5 Power, U1 TL074

Commit message: Switch 348 output buffer to kicad6
Parts:
- J1, J2, J3, J4: symbol WireConnections:Wire_24AWG_Stranded -> Wire_Connections:Wire_24AWG_Stranded
- RV1, RV2, RV3, RV4: symbol Device:R_POT_TRIM -> Device:R_Potentiometer_Trim
Changed lines of the file:
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@@
     (pin "1")
   )
-  (symbol (lib_id "Device:R_POT_TRIM") (at 64.77 69.85 90) (unit 1)
+  (symbol (lib_id "Device:R_Potentiometer_Trim") (at 64.77 69.85 90) (unit 1)
     (in_bom yes) (on_board yes)
     (property "Reference" "RV1" (id 0) (at 64.77 75.1078 90))
@@
     (pin "1")
   )
-  (symbol (lib_id "WireConnections:Wire_24AWG_Stranded") (at 36.83 80.01 0) (unit 1)
+  (symbol (lib_id "Wire_Connections:Wire_24AWG_Stranded") (at 36.83 80.01 0) (unit 1)
     (in_bom yes) (on_board yes)
     (property "Reference" "J1" (id 0) (at 37.6682 74.8792 0))
@@
     (pin "1")
   )
-  (symbol (lib_id "WireConnections:Wire_24AWG_Stranded") (at 124.46 85.09 0) (mirror y) (unit 1)
+  (symbol (lib_id "Wire_Connections:Wire_24AWG_Stranded") (at 124.46 85.09 0) (mirror y) (unit 1)
     (in_bom yes) (on_board yes)
     (property "Reference" "J3" (id 0) (at 123.6218 79.9592 0))
@@
     (pin "2")
   )
-  (symbol (lib_id "WireConnections:Wire_24AWG_Stranded") (at 128.27 149.86 0) (mirror y) (unit 1)
+  (symbol (lib_id "Wire_Connections:Wire_24AWG_Stranded") (at 128.27 149.86 0) (mirror y) (unit 1)
     (in_bom yes) (on_board yes)
     (property "Reference" "J4" (id 0) (at 127.4318 144.7292 0))
@@
     (pin "1")
   )
-  (symbol (lib_id "WireConnections:Wire_24AWG_Stranded") (at 40.64 144.78 0) (unit 1)
+  (symbol (lib_id "Wire_Connections:Wire_24AWG_Stranded") (at 40.64 144.78 0) (unit 1)
     (in_bom yes) (on_board yes)
     (property "Reference" "J2" (id 0) (at 41.4782 139.6492 0))
@@
     (pin "1")
   )
-  (symbol (lib_id "Device:R_POT_TRIM") (at 87.63 50.8 270) (unit 1)
+  (symbol (lib_id "Device:R_Potentiometer_Trim") (at 87.63 50.8 270) (unit 1)
     (in_bom yes) (on_board yes)
     (property "Reference" "RV3" (id 0) (at 87.63 45.5422 90))
@@
     (pin "2")
   )
-  (symbol (lib_id "Device:R_POT_TRIM") (at 91.44 115.57 270) (unit 1)
+  (symbol (lib_id "Device:R_Potentiometer_Trim") (at 91.44 115.57 270) (unit 1)
     (in_bom yes) (on_board yes)
     (property "Reference" "RV4" (id 0) (at 91.44 110.3122 90))
@@
     (pin "1")
   )
-  (symbol (lib_id "Device:R_POT_TRIM") (at 68.58 134.62 90) (unit 1)
+  (symbol (lib_id "Device:R_Potentiometer_Trim") (at 68.58 134.62 90) (unit 1)
     (in_bom yes) (on_board yes)
     (property "Reference" "RV2" (id 0) (at 68.58 139.8778 90))
