File: cgs-attenuverter-board/cgs-attenuverter-board.kicad_pcb (KiCad board)
At the start: 2 copper layers, 50.3 x 39.4 mm, 22 parts, among them J5 Power, U1 TL072

Commit message: Updating ordered boards
Other:
- rule pad_to_mask_clearance: 0.0508 -> 0

Commit message: Updates to attenuverter board
Parts:
- moved C1 18.0 mm to (143.3, 90.4)
- moved C2 17.8 mm to (161.3, 95.4)
- renumbered IN1 to J1, IN2 to J2, OUT1 to J3, OUT2 to J4
Connections:
- J5 pad 1: +12V -> -12V
- J5 pad 3: -12V -> +12V
- U1 pad 4: +12V -> -12V
- U1 pad 8: -12V -> +12V
Routing:
- net +12V: track 27.9 -> 37.0 mm
- net -12V: track 36.5 -> 28.0 mm
- added copper zone on F.Cu, net GND
- removed copper zone on F.Cu, net (none)
Other:
- board text added: "+V"
- board text added: "-V"
- board text added: "ATTV1"
- board text added: "ATTV2"
- board text added: "IN1"
- board text added: "IN2"
- board text added: "OUT1"
- board text added: "OUT2"
- board text added: "Precision Attenuverter r02"
- board text removed: "Precision Attenuverter r01"
