File: cgs-attenuverter-board/cgs-attenuverter-board.sch (KiCad schematic (older format))
At the start: 22 parts, among them J1 IN, J2 IN, J3 OUT, J4 OUT, J5 Power, U1 TL072

Commit message: Updates to attenuverter board
Connections:
- net +12V: now also J5.3 (Pin_3), U1.8 (V+); no longer J5.1 (Pin_1), U1.4 (V-)
- net -12V: now also J5.1 (Pin_1), U1.4 (V-); no longer J5.3 (Pin_3), U1.8 (V+)
Changed lines of the file:
@@
 F 3 "~" H 6500 2950 50  0001 C CNN
 	1    6500 2950
-	1    0    0    -1
+	1    0    0    1
 $EndComp
 $Comp
@@
 L Amplifier_Operational:TL072 U1
 U 3 1 622C3BA8
-P 6650 4250
-F 0 "U1" H 6463 4204 50  0000 R CNN
-F 1 "TL072" H 6463 4295 50  0000 R CNN
-F 2 "Package_DIP:DIP-8_W7.62mm_Socket" H 6650 4250 50  0001 C CNN
-F 3 "http://www.ti.com/lit/ds/symlink/tl071.pdf" H 6650 4250 50  0001 C CNN
-	3    6650 4250
-	1    0    0    1
+P 6450 4250
+F 0 "U1" H 6263 4204 50  0000 R CNN
+F 1 "TL072" H 6263 4295 50  0000 R CNN
+F 2 "Package_DIP:DIP-8_W7.62mm_Socket" H 6450 4250 50  0001 C CNN
+F 3 "http://www.ti.com/lit/ds/symlink/tl071.pdf" H 6450 4250 50  0001 C CNN
+	3    6450 4250
+	-1   0    0    -1
 $EndComp
 $Comp
