File: 4u-spring-reverb/4u-spring-reverb.kicad_pcb (KiCad board)
At the start: 2 copper layers, 50.8 x 111.8 mm, 65 parts, among them J1 IN1, J10 MIX_MAIN, J11 AUDIO_IO_MAIN, J12 AUDIO_IO_CTRL, J2 REV_RETURN, J3 IN2, J4 OUT, J5 REV_SEND, J6 TILT_MAIN, J7 TILT_CTRL, J8 Conn_01x04_Male, J9 MIX_CTRL, U1 TL072, U2 NE5532, U3 TL072

Commit message: Updating spring reverb
Routing:
- net +12V: track 104.3 -> 108.2 mm
- net /AUDIO_OUT_MAIN: track 25.4 -> 28.7 mm
- net /TILT_LO_MAIN: track 27.0 -> 26.0 mm
Changed lines of the file:
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@@
     (thickness 1.6)
     (drawings 55)
-    (tracks 237)
+    (tracks 244)
     (zones 0)
     (modules 65)
@@
       (psnegative false)
       (psa4output false)
-      (plotreference true)
+      (plotreference false)
       (plotvalue false)
       (plotinvisibletext false)
@@
     (pad 2 thru_hole oval (at 2.54 0) (size 1.74 2.19) (drill 1.19) (layers *.Cu *.Mask)
       (net 7 GND))
-    (pad 1 thru_hole roundrect (at 0 0) (size 1.74 2.19) (drill 1.19) (layers *.Cu *.Mask) (roundrect_rratio 0.143678)
+    (pad 1 thru_hole roundrect (at 0 0) (size 1.74 2.19) (drill 1.19) (layers *.Cu *.Mask) (roundrect_rratio 0.1436775862068966)
       (net 29 "Net-(D1-Pad2)"))
     (model ${KISYS3DMOD}/Connector_Molex.3dshapes/Molex_KK-254_AE-6410-04A_1x04_P2.54mm_Vertical.wrl
@@
   (segment (start 139.112 119.38) (end 137.668 119.38) (width 1.27) (layer F.Cu) (net 8))
   (segment (start 135.128 58.42) (end 138.176 58.42) (width 1.27) (layer F.Cu) (net 8))
-  (segment (start 137.034999 59.561001) (end 138.176 58.42) (width 1.27) (layer F.Cu) (net 8))
   (segment (start 139.112 90.002722) (end 137.034999 87.925721) (width 1.27) (layer F.Cu) (net 8))
-  (segment (start 137.034999 87.925721) (end 137.034999 59.561001) (width 1.27) (layer F.Cu) (net 8))
   (segment (start 139.112 119.38) (end 139.112 90.002722) (width 1.27) (layer F.Cu) (net 8))
+  (segment (start 139.650723 75.001001) (end 138.579279 75.001001) (width 1.27) (layer F.Cu) (net 8))
+  (segment (start 140.674001 76.024279) (end 139.650723 75.001001) (width 1.27) (layer F.Cu) (net 8))
+  (segment (start 135.128 71.549722) (end 135.128 58.42) (width 1.27) (layer F.Cu) (net 8))
+  (segment (start 140.674001 77.645721) (end 140.674001 76.024279) (width 1.27) (layer F.Cu) (net 8))
+  (segment (start 137.034999 81.284723) (end 140.674001 77.645721) (width 1.27) (layer F.Cu) (net 8))
+  (segment (start 138.579279 75.001001) (end 135.128 71.549722) (width 1.27) (layer F.Cu) (net 8))
+  (segment (start 137.034999 87.925721) (end 137.034999 81.284723) (width 1.27) (layer F.Cu) (net 8))
   (segment (start 148.55 139.7) (end 145.248 136.398) (width 1.27) (layer F.Cu) (net 9))
   (segment (start 148.59 139.7) (end 148.55 139.7) (width 1.27) (layer F.Cu) (net 9))
@@
   (segment (start 145.796 48.514) (end 147.32 46.99) (width 1.27) (layer F.Cu) (net 9))
   (segment (start 145.796 50.8) (end 145.796 48.514) (width 1.27) (layer F.Cu) (net 9))
-  (segment (start 144.106999 74.206001) (end 144.106999 52.489001) (width 1.27) (layer F.Cu) (net 9))
-  (segment (start 140.969999 77.343001) (end 144.106999 74.206001) (width 1.27) (layer F.Cu) (net 9))
-  (segment (start 140.969999 104.139999) (end 140.969999 77.343001) (width 1.27) (layer F.Cu) (net 9))
-  (segment (start 144.106999 52.489001) (end 145.796 50.8) (width 1.27) (layer F.Cu) (net 9))
-  (segment (start 141.986 105.156) (end 140.969999 104.139999) (width 1.27) (layer F.Cu) (net 9))
+  (segment (start 140.969999 104.139999) (end 141.986 105.156) (width 1.27) (layer F.Cu) (net 9))
+  (segment (start 142.93849 78.970788) (end 140.969999 80.939279) (width 1.27) (layer F.Cu) (net 9))
+  (segment (start 140.969999 80.939279) (end 140.969999 104.139999) (width 1.27) (layer F.Cu) (net 9))
+  (segment (start 142.93849 75.586) (end 142.93849 78.970788) (width 1.27) (layer F.Cu) (net 9))
+  (segment (start 144.106999 74.417491) (end 142.93849 75.586) (width 1.27) (layer F.Cu) (net 9))
+  (segment (start 144.106999 52.489001) (end 144.106999 74.417491) (width 1.27) (layer F.Cu) (net 9))
+  (segment (start 145.796 50.8) (end 144.106999 52.489001) (width 1.27) (layer F.Cu) (net 9))
   (segment (start 148.336 66.802) (end 149.098 66.04) (width 0.635) (layer B.Cu) (net 10))
   (segment (start 145.796 66.802) (end 148.336 66.802) (width 0.635) (layer B.Cu) (net 10))
@@
   (segment (start 130.937 101.727) (end 129.794 102.87) (width 0.635) (layer B.Cu) (net 13))
   (segment (start 134.62 101.727) (end 130.937 101.727) (width 0.635) (layer B.Cu) (net 13))
-  (segment (start 132.715 94.869) (end 129.794 97.79) (width 0.635) (layer B.Cu) (net 14))
-  (segment (start 133.731 94.869) (end 132.715 94.869) (width 0.635) (layer B.Cu) (net 14))
-  (segment (start 128.372499 99.211501) (end 129.794 97.79) (width 0.635) (layer B.Cu) (net 14))
-  (segment (start 128.372499 115.418499) (end 128.372499 99.211501) (width 0.635) (layer B.Cu) (net 14))
-  (segment (start 129.794 116.84) (end 128.372499 115.418499) (width 0.635) (layer B.Cu) (net 14))
-  (segment (start 130.937 87.503) (end 129.54 88.9) (width 0.635) (layer B.Cu) (net 15))
-  (segment (start 134.112 87.503) (end 130.937 87.503) (width 0.635) (layer B.Cu) (net 15))
+  (segment (start 132.931001 113.702999) (end 129.794 116.84) (width 0.635) (layer F.Cu) (net 14))
+  (segment (start 132.931001 95.668999) (end 132.931001 113.702999) (width 0.635) (layer F.Cu) (net 14))
+  (segment (start 133.731 94.869) (end 132.931001 95.668999) (width 0.635) (layer F.Cu) (net 14))
+  (segment (start 130.81 97.79) (end 133.731 94.869) (width 0.635) (layer F.Cu) (net 14))
+  (segment (start 129.794 97.79) (end 130.81 97.79) (width 0.635) (layer F.Cu) (net 14))
   (segment (start 134.112 83.693) (end 134.112 87.503) (width 0.635) (layer F.Cu) (net 15))
+  (segment (start 132.715 88.9) (end 134.112 87.503) (width 0.635) (layer F.Cu) (net 15))
+  (segment (start 129.54 88.9) (end 132.715 88.9) (width 0.635) (layer F.Cu) (net 15))
   (segment (start 143.75237 76.835) (end 138.985 76.835) (width 0.635) (layer B.Cu) (net 16))
   (segment (start 147.447 80.52963) (end 143.75237 76.835) (width 0.635) (layer B.Cu) (net 16))
   (segment (start 147.447 81.661) (end 147.447 80.52963) (width 0.635) (layer B.Cu) (net 16))
   (segment (start 129.54 86.36) (end 129.768501 86.131499) (width 0.635) (layer B.Cu) (net 16))
-  (segment (start 137.613499 78.206501) (end 138.985 76.835) (width 0.635) (layer B.Cu) (net 16))
-  (segment (start 130.784501 81.434677) (end 134.012677 78.206501) (width 0.635) (layer B.Cu) (net 16))
-  (segment (start 134.012677 78.206501) (end 137.613499 78.206501) (width 0.635) (layer B.Cu) (net 16))
-  (segment (start 130.784501 85.115499) (end 130.784501 81.434677) (width 0.635) (layer B.Cu) (net 16))
-  (segment (start 129.54 86.36) (end 130.784501 85.115499) (width 0.635) (layer B.Cu) (net 16))
+  (segment (start 138.985 77.293822) (end 138.985 76.835) (width 0.635) (layer F.Cu) (net 16))
+  (segment (start 129.54 84.875) (end 132.779499 81.635501) (width 0.635) (layer F.Cu) (net 16))
+  (segment (start 134.643321 81.635501) (end 138.985 77.293822) (width 0.635) (layer F.Cu) (net 16))
+  (segment (start 132.779499 81.635501) (end 134.643321 81.635501) (width 0.635) (layer F.Cu) (net 16))
+  (segment (start 129.54 86.36) (end 129.54 84.875) (width 0.635) (layer F.Cu) (net 16))
   (segment (start 132.668 109.3) (end 134.366 110.998) (width 0.635) (layer B.Cu) (net 17))
   (segment (start 130.302 109.3) (end 132.668 109.3) (width 0.635) (layer B.Cu) (net 17))
-  (segment (start 131.215501 108.386499) (end 131.215501 93.115501) (width 0.635) (layer F.Cu) (net 17))
-  (segment (start 131.215501 93.115501) (end 129.54 91.44) (width 0.635) (layer F.Cu) (net 17))
-  (segment (start 130.302 109.3) (end 131.215501 108.386499) (width 0.635) (layer F.Cu) (net 17))
+  (segment (start 128.372499 92.607501) (end 129.54 91.44) (width 0.635) (layer F.Cu) (net 17))
+  (segment (start 128.372499 107.370499) (end 128.372499 92.607501) (width 0.635) (layer F.Cu) (net 17))
+  (segment (start 130.302 109.3) (end 128.372499 107.370499) (width 0.635) (layer F.Cu) (net 17))
   (segment (start 114.367501 107.628499) (end 121.666 100.33) (width 0.635) (layer B.Cu) (net 18))
   (segment (start 113.231501 107.628499) (end 114.367501 107.628499) (width 0.635) (layer B.Cu) (net 18))
@@
   (segment (start 138.176 48.514) (end 139.7 46.99) (width 0.635) (layer F.Cu) (net 41))
   (segment (start 138.176 50.8) (end 138.176 48.514) (width 0.635) (layer F.Cu) (net 41))
-  (zone (net 7) (net_name GND) (layer F.Cu) (hatch edge 0.508)
+  (zone (net 24) (net_name GND1) (layer F.Cu) (hatch edge 0.508)
     (connect_pads (clearance 0.508))
     (min_thickness 0.254)
@@
     (polygon
       (pts
-        (xy 151.257 149.987) (xy 126.873 149.987) (xy 126.873 37.973) (xy 151.257 37.973)
+        (xy 124.587 149.987) (xy 100.203 149.987) (xy 100.203 37.973) (xy 124.587 37.973)
       )
     )
   )
-  (zone (net 24) (net_name GND1) (layer F.Cu) (hatch edge 0.508)
+  (zone (net 24) (net_name GND1) (layer B.Cu) (hatch edge 0.508)
     (connect_pads (clearance 0.508))
     (min_thickness 0.254)
@@
     )
   )
-  (zone (net 7) (net_name GND) (layer B.Cu) (hatch edge 0.508)
+  (zone (net 7) (net_name GND) (layer F.Cu) (hatch edge 0.508)
     (connect_pads (clearance 0.508))
     (min_thickness 0.254)
@@
     (polygon
       (pts
-        (xy 151.257 149.987) (xy 126.873 149.987) (xy 126.873 37.973) (xy 151.257 37.973)
+        (xy 151.1 149.9) (xy 126.9 149.9) (xy 126.9 38) (xy 151.2 38)
       )
     )
   )
-  (zone (net 24) (net_name GND1) (layer B.Cu) (hatch edge 0.508)
+  (zone (net 7) (net_name GND) (layer B.Cu) (hatch edge 0.508)
     (connect_pads (clearance 0.508))
     (min_thickness 0.254)
@@
     (polygon
       (pts
-        (xy 124.587 149.987) (xy 100.203 149.987) (xy 100.203 37.973) (xy 124.587 37.973)
+        (xy 151.1 149.9) (xy 126.9 149.9) (xy 126.9 38) (xy 151.2 38)
       )
     )
