File: 4u-spring-reverb/4u-spring-reverb.sch (KiCad schematic (older format))
At the start: 55 parts, among them J1 IN1, J10 MIX_MAIN, J11 AUDIO_IO_MAIN, J12 AUDIO_IO_CTRL, J2 REV_RETURN, J3 IN2, J4 OUT, J5 REV_SEND, J6 TILT_MAIN, J7 TILT_CTRL, J8 Conn_01x04_Male, J9 MIX_CTRL, U1 TL072, U2 NE5532, U3 TL072

Commit message: Updating spring reverb
Other:
- note added: "R2 and R3 set recovery level\nR2 should be smaller than output coil impedance\n2250/2575r: R2 = 22r R3 = 22k\nIncrease R3 for stronger output,\nreduce R3 if circuit distorts even when\nspring drive is set low"
- note added: "Values for R14:\n800r tank: R14 = 2k\n150r tank: R14 = 470r\nor use 10k trimmer"
- note removed: "R4 and R6 set recovery level\nR4 should be smaller than output coil impedance\n2250/2575r: R4 = 22r R6 = 22k\nIncrease R6 for stronger output,\nreduce R6 if circuit distorts even when\nspring drive is set low"
- note removed: "Values for R2:\n800r tank: R2 = 2k\n150r tank: R2 = 470r\nor use 10k trimmer"
Changed lines of the file:
@@
 $EndComp
 Text Notes 9050 3500 0    50   ~ 0
-Values for R2:\n800r tank: R2 = 2k\n150r tank: R2 = 470r\nor use 10k trimmer
+Values for R14:\n800r tank: R14 = 2k\n150r tank: R14 = 470r\nor use 10k trimmer
 Text Notes 2650 6750 0    50   ~ 0
-R4 and R6 set recovery level\nR4 should be smaller than output coil impedance\n2250/2575r: R4 = 22r R6 = 22k\nIncrease R6 for stronger output,\nreduce R6 if circuit distorts even when\nspring drive is set low
+R2 and R3 set recovery level\nR2 should be smaller than output coil impedance\n2250/2575r: R2 = 22r R3 = 22k\nIncrease R3 for stronger output,\nreduce R3 if circuit distorts even when\nspring drive is set low
 Text Label 5650 2050 0    50   ~ 0
 AUDIO_MIX
