File: serge-vcfs/serge-vcfs.kicad_pcb (KiCad board)
At the start: 2 copper layers, 0 parts

Commit message: Fixing issue with vcfs
Parts:
- added C1: 10uf, rumblesan-footprints:CP_Radial_D5.0mm_P2.50mm, F.Cu at (134.6, 35.6)
- added C10: 100nF, rumblesan-footprints:C_Rect_L7.0mm_W3.5mm_P5.00mm, F.Cu at (127.8, 35.8)
- added C11: 100nF, rumblesan-footprints:C_Rect_L7.0mm_W3.5mm_P5.00mm, F.Cu at (109.7, 40.4)
- added C12: 100nF, rumblesan-footprints:C_Rect_L7.0mm_W3.5mm_P5.00mm, F.Cu at (136.6, 166.4)
- added C13: 100nF, rumblesan-footprints:C_Rect_L7.0mm_W3.5mm_P5.00mm, F.Cu at (113.5, 133.3)
- added C14: 100nF, rumblesan-footprints:C_Rect_L7.0mm_W3.5mm_P5.00mm, F.Cu at (127.8, 144.8)
- added C15: 100nF, rumblesan-footprints:C_Rect_L7.0mm_W3.5mm_P5.00mm, F.Cu at (116.6, 163.9)
- added C16: 100nF, rumblesan-footprints:C_Rect_L7.0mm_W3.5mm_P5.00mm, F.Cu at (117.9, 82.3)
- added C2: 10uF, rumblesan-footprints:CP_Radial_D5.0mm_P2.50mm, F.Cu at (129.0, 94.5)
- added C3: 10uF, rumblesan-footprints:CP_Radial_D5.0mm_P2.50mm, F.Cu at (102.9, 38.4)
- added C4: 220pF, rumblesan-footprints:C_Axial_L12.0mm_D5.0mm_P15.00mm_Horizontal, F.Cu at (129.5, 62.5)
- added C5: 15pF, rumblesan-footprints:C_Rect_L7.0mm_W3.5mm_P5.00mm, F.Cu at (120.0, 68.3)
- added C6: 15pF, rumblesan-footprints:C_Rect_L7.0mm_W3.5mm_P5.00mm, F.Cu at (126.2, 56.4)
- added C7: 220pF, rumblesan-footprints:C_Axial_L12.0mm_D5.0mm_P15.00mm_Horizontal, F.Cu at (112.5, 61.2)
- added C8: 100nF, rumblesan-footprints:C_Rect_L7.0mm_W3.5mm_P5.00mm, F.Cu at (111.3, 93.7)
- added C9: 220pF, rumblesan-footprints:C_Rect_L7.0mm_W3.5mm_P5.00mm, F.Cu at (116.3, 156.0)
- added D1: 1n4148, rumblesan-footprints:Diode_THT_P7.62mm_Horizontal, F.Cu at (116.8, 126.7)
- added D2: 1n4148, rumblesan-footprints:Diode_THT_P7.62mm_Horizontal, F.Cu at (111.8, 144.8)
- added D3: 1n4148, rumblesan-footprints:Diode_THT_P7.62mm_Horizontal, F.Cu at (138.9, 144.0)
- added H1: MountingScrew_M3_Flathead, MountingHole:MountingHole_3.2mm_M3, F.Cu at (138.7, 100.6)
- added H2: MountingScrew_M3_Flathead, MountingHole:MountingHole_3.2mm_M3, F.Cu at (52.3, 100.6)
- added J1: In 1, rumblesan-footprints:BananaJack_THT_JohnsonCinch_108-09, F.Cu at (57.4, 89.4)
- added J10: V/Oct, rumblesan-footprints:BananaJack_THT_JohnsonCinch_108-09, F.Cu at (82.8, 95.8)
- added J11: VC Freq, rumblesan-footprints:BananaJack_THT_JohnsonCinch_108-09, F.Cu at (82.8, 114.8)
- added J12: HP Out, rumblesan-footprints:BananaJack_THT_JohnsonCinch_108-09, F.Cu at (82.8, 38.6)
- added J13: BP Out, rumblesan-footprints:BananaJack_THT_JohnsonCinch_108-09, F.Cu at (57.4, 38.6)
- added J14: Conn_01x04_Female, Connector_PinHeader_2.54mm:PinHeader_1x04_P2.54mm_Vertical, B.Cu at (75.4, 57.4)
- added J15: Conn_01x04_Male, Connector_PinSocket_2.54mm:PinSocket_1x04_P2.54mm_Vertical, B.Cu at (115.6, 57.4)
- added J16: LOW Out, rumblesan-footprints:BananaJack_THT_JohnsonCinch_108-09, F.Cu at (82.8, 57.7)
- added J17: Power, rumblesan-footprints:Molex_KK-254_AE-6410-04A_1x04_P2.54mm_Vertical, F.Cu at (114.8, 38.1)
- added J18: Conn_01x02_Female, Connector_PinSocket_2.54mm:PinSocket_1x02_P2.54mm_Vertical, B.Cu at (81.0, 129.5)
- added J19: Conn_01x02_Male, Connector_PinHeader_2.54mm:PinHeader_1x02_P2.54mm_Vertical, B.Cu at (110.0, 129.5)
- added J2: In 2, rumblesan-footprints:BananaJack_THT_JohnsonCinch_108-09, F.Cu at (82.8, 76.7)
- added J3: Conn_01x02_Female, Connector_PinHeader_2.54mm:PinHeader_1x02_P2.54mm_Vertical, B.Cu at (71.6, 100.6)
- added J4: Conn_01x04_Female, Connector_PinHeader_2.54mm:PinHeader_1x04_P2.54mm_Vertical, B.Cu at (91.7, 163.1)
- added J5: Conn_01x02_Male, Connector_PinSocket_2.54mm:PinSocket_1x02_P2.54mm_Vertical, B.Cu at (119.4, 100.6)
- added J6: Conn_01x04_Female, Connector_PinHeader_2.54mm:PinHeader_1x04_P2.54mm_Vertical, B.Cu at (48.5, 168.1)
- added J7: Conn_01x04_Male, Connector_PinSocket_2.54mm:PinSocket_1x04_P2.54mm_Vertical, B.Cu at (99.3, 163.1)
- added J8: Conn_01x04_Male, Connector_PinSocket_2.54mm:PinSocket_1x04_P2.54mm_Vertical, B.Cu at (142.5, 168.1)
- added J9: VC Slope, rumblesan-footprints:BananaJack_THT_JohnsonCinch_108-09, F.Cu at (57.4, 114.8)
- added Q1: 2N3904, Package_TO_SOT_THT:TO-92_Inline, F.Cu at (134.9, 110.0)
- added Q2: 2N3904, Package_TO_SOT_THT:TO-92_Inline, F.Cu at (133.9, 126.5)
- added Q3: 2N3904, Package_TO_SOT_THT:TO-92_Inline, F.Cu at (108.7, 109.7)
- added R1: 330r, rumblesan-footprints:R_Axial_DIN0207_L6.3mm_D2.5mm_P7.62mm_Horizontal, F.Cu at (112.0, 79.0)
- added R10: 47k, rumblesan-footprints:R_Axial_DIN0207_L6.3mm_D2.5mm_P7.62mm_Horizontal, F.Cu at (125.0, 61.7)
- added R11: 330k, rumblesan-footprints:R_Axial_DIN0207_L6.3mm_D2.5mm_P7.62mm_Horizontal, F.Cu at (124.5, 129.8)
- added R12: 820r, rumblesan-footprints:R_Axial_DIN0207_L6.3mm_D2.5mm_P7.62mm_Horizontal, F.Cu at (127.8, 141.0)
- added R13: 22k, rumblesan-footprints:R_Axial_DIN0207_L6.3mm_D2.5mm_P7.62mm_Horizontal, F.Cu at (124.5, 111.3)
- added R14: 33k, rumblesan-footprints:R_Axial_DIN0207_L6.3mm_D2.5mm_P7.62mm_Horizontal, F.Cu at (107.4, 91.4)
- added R15: 22k, rumblesan-footprints:R_Axial_DIN0207_L6.3mm_D2.5mm_P7.62mm_Horizontal, F.Cu at (131.3, 150.4)
- added R16: 475r, rumblesan-footprints:R_Axial_DIN0207_L6.3mm_D2.5mm_P7.62mm_Horizontal, F.Cu at (124.5, 117.3)
- added R17: 475r, rumblesan-footprints:R_Axial_DIN0207_L6.3mm_D2.5mm_P7.62mm_Horizontal, F.Cu at (116.8, 105.2)
- added R18: 6k8, rumblesan-footprints:R_Axial_DIN0207_L6.3mm_D2.5mm_P7.62mm_Horizontal, F.Cu at (130.8, 120.4)
- added R19: 6k8, rumblesan-footprints:R_Axial_DIN0207_L6.3mm_D2.5mm_P7.62mm_Horizontal, F.Cu at (124.5, 120.4)
- added R2: 220k, rumblesan-footprints:R_Axial_DIN0207_L6.3mm_D2.5mm_P7.62mm_Horizontal, F.Cu at (117.3, 74.9)
- added R20: 47k, rumblesan-footprints:R_Axial_DIN0207_L6.3mm_D2.5mm_P7.62mm_Horizontal, F.Cu at (138.9, 140.7)
- added R21: 15k, rumblesan-footprints:R_Axial_DIN0207_L6.3mm_D2.5mm_P7.62mm_Horizontal, F.Cu at (138.9, 147.3)
- added R22: 33k, rumblesan-footprints:R_Axial_DIN0207_L6.3mm_D2.5mm_P7.62mm_Horizontal, F.Cu at (138.9, 156.5)
- added R23: 1M0, rumblesan-footprints:R_Axial_DIN0207_L6.3mm_D2.5mm_P7.62mm_Horizontal, F.Cu at (131.3, 159.5)
- added R24: 22k, rumblesan-footprints:R_Axial_DIN0207_L6.3mm_D2.5mm_P7.62mm_Horizontal, F.Cu at (128.0, 148.8)
- added R25: 390r, rumblesan-footprints:R_Axial_DIN0207_L6.3mm_D2.5mm_P7.62mm_Horizontal, F.Cu at (124.5, 114.3)
- added R26: 15k, rumblesan-footprints:R_Axial_DIN0207_L6.3mm_D2.5mm_P7.62mm_Horizontal, F.Cu at (131.3, 153.4)
- added R27: 330k, rumblesan-footprints:R_Axial_DIN0207_L6.3mm_D2.5mm_P7.62mm_Horizontal, F.Cu at (128.0, 154.9)
- added R28: 2k, rumblesan-footprints:R_Axial_DIN0207_L6.3mm_D2.5mm_P7.62mm_Horizontal, F.Cu at (128.0, 151.9)
- added R29: 220k, rumblesan-footprints:R_Axial_DIN0207_L6.3mm_D2.5mm_P7.62mm_Horizontal, F.Cu at (131.3, 162.6)
- added R3: 220k, rumblesan-footprints:R_Axial_DIN0207_L6.3mm_D2.5mm_P7.62mm_Horizontal, F.Cu at (117.3, 71.9)
- added R30: 470k, rumblesan-footprints:R_Axial_DIN0207_L6.3mm_D2.5mm_P7.62mm_Horizontal, F.Cu at (131.3, 170.2)
- added R31: 1M, rumblesan-footprints:R_Axial_DIN0207_L6.3mm_D2.5mm_P7.62mm_Horizontal, F.Cu at (131.3, 179.3)
- added R32: 330k, rumblesan-footprints:R_Axial_DIN0207_L6.3mm_D2.5mm_P7.62mm_Horizontal, F.Cu at (138.9, 173.2)
- added R33: 330k, rumblesan-footprints:R_Axial_DIN0207_L6.3mm_D2.5mm_P7.62mm_Horizontal, F.Cu at (131.3, 176.3)
- added R34: 22k, rumblesan-footprints:R_Axial_DIN0207_L6.3mm_D2.5mm_P7.62mm_Horizontal, F.Cu at (102.6, 168.1)
- added R35: 22k, rumblesan-footprints:R_Axial_DIN0207_L6.3mm_D2.5mm_P7.62mm_Horizontal, F.Cu at (110.2, 165.1)
- added R36: 100k, rumblesan-footprints:R_Axial_DIN0207_L6.3mm_D2.5mm_P7.62mm_Horizontal, F.Cu at (110.2, 162.1)
- added R37: 22k, rumblesan-footprints:R_Axial_DIN0207_L6.3mm_D2.5mm_P7.62mm_Horizontal, F.Cu at (74.9, 86.4)
- added R38: 22k, rumblesan-footprints:R_Axial_DIN0207_L6.3mm_D2.5mm_P7.62mm_Horizontal, F.Cu at (67.3, 89.8)
- added R39: 47k, rumblesan-footprints:R_Axial_DIN0207_L6.3mm_D2.5mm_P7.62mm_Horizontal, F.Cu at (88.0, 136.3)
- added R4: 100k, rumblesan-footprints:R_Axial_DIN0207_L6.3mm_D2.5mm_P7.62mm_Horizontal, F.Cu at (130.0, 97.8)
- added R40: 82k, rumblesan-footprints:R_Axial_DIN0207_L6.3mm_D2.5mm_P7.62mm_Horizontal, F.Cu at (110.2, 171.2)
- added R5: 100k, rumblesan-footprints:R_Axial_DIN0207_L6.3mm_D2.5mm_P7.62mm_Horizontal, F.Cu at (130.0, 100.8)
- added R6: 220k, rumblesan-footprints:R_Axial_DIN0207_L6.3mm_D2.5mm_P7.62mm_Horizontal, F.Cu at (125.0, 78.0)
- added R7: 330r, rumblesan-footprints:R_Axial_DIN0207_L6.3mm_D2.5mm_P7.62mm_Horizontal, F.Cu at (118.6, 52.8)
- added R8: 330r, rumblesan-footprints:R_Axial_DIN0207_L6.3mm_D2.5mm_P7.62mm_Horizontal, F.Cu at (118.6, 49.8)
- added R9: 47k, rumblesan-footprints:R_Axial_DIN0207_L6.3mm_D2.5mm_P7.62mm_Horizontal, F.Cu at (117.3, 64.8)
- added RV1: 50kB, rumblesan-footprints:Potentiometer_Alpha_RD901F-40-00D_Single_Vertical_CircularHoles, F.Cu at (57.4, 64.0)
- added RV2: 50kB, rumblesan-footprints:Potentiometer_Alpha_RD901F-40-00D_Single_Vertical_CircularHoles, F.Cu at (57.4, 172.0)
- added RV3: 10k, rumblesan-footprints:Potentiometer_THT_Bourns_3306P_Vertical, F.Cu at (114.0, 177.0)
- added RV4: 50kB, rumblesan-footprints:Potentiometer_Alpha_RD901F-40-00D_Single_Vertical_CircularHoles, F.Cu at (57.4, 143.4)
- added RV5: 50kB, rumblesan-footprints:Potentiometer_Alpha_RD901F-40-00D_Single_Vertical_CircularHoles, F.Cu at (82.8, 172.0)
- added RV6: 50kB, rumblesan-footprints:Potentiometer_Alpha_RD901F-40-00D_Single_Vertical_CircularHoles, F.Cu at (82.8, 143.4)
- added U1: TL074, rumblesan-footprints:DIP-14_W7.62mm_Socket, F.Cu at (120.4, 158.8)
- added U2: TL072, rumblesan-footprints:DIP-8_W7.62mm_Socket, F.Cu at (122.9, 93.7)
- added U3: CGS108_Serge_Gain_Cell, rumblesan-footprints:Serge_GainCell_Vertical, F.Cu at (106.9, 51.1)
- added U4: CGS108_Serge_Gain_Cell, rumblesan-footprints:Serge_GainCell_Vertical, F.Cu at (141.2, 50.8)
- added U5: TL072, rumblesan-footprints:DIP-8_W7.62mm_Socket, F.Cu at (116.8, 141.0)
- added mouse-bite-2.54mm-slot: VAL**, rumblesan-footprints:mouse-bite-2.54mm-slot, F.Cu at (95.5, 169.7)
- added mouse-bite-2.54mm-slot: VAL**, rumblesan-footprints:mouse-bite-2.54mm-slot, F.Cu at (95.5, 139.4)
- added mouse-bite-2.54mm-slot: VAL**, rumblesan-footprints:mouse-bite-2.54mm-slot, F.Cu at (95.5, 104.9)
- added mouse-bite-2.54mm-slot: VAL**, rumblesan-footprints:mouse-bite-2.54mm-slot, F.Cu at (95.5, 67.3)
- added mouse-bite-2.54mm-slot: VAL**, rumblesan-footprints:mouse-bite-2.54mm-slot, F.Cu at (95.5, 40.1)
Routing:
- net -12V: track 0.00 -> 268.2 mm
- net +12V: track 0.00 -> 226.6 mm
- net /FREQ-CV-1: track 0.00 -> 95.3 mm
- net /FREQ-CV-2: track 0.00 -> 78.2 mm
- net +12VA: track 0.00 -> 77.4 mm
- net /VOCT_IO: track 0.00 -> 75.3 mm
- net /VC_SLOPE_IO: track 0.00 -> 66.2 mm
- net Net-(R16-Pad2): track 0.00 -> 56.1 mm
- net Net-(Q1-Pad2): track 0.00 -> 51.4 mm
- net Net-(C4-Pad1): track 0.00 -> 43.8 mm
- net /VC_FREQ_CCW_MAIN: track 0.00 -> 39.7 mm
- net /IN_1_IO: track 0.00 -> 36.8 mm
- net Net-(C5-Pad2): track 0.00 -> 36.7 mm
- net /IN_2_IO: track 0.00 -> 34.6 mm
- net Net-(C2-Pad2): track 0.00 -> 33.9 mm
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- added copper zone on B.Cu, net GND
- added copper zone on F.Cu, net GND
- added copper zone on B.Cu, net GNDA
- added copper zone on F.Cu, net GNDA
Other:
- board outline added: 99.1 x 150.6 mm
- board text added: "1V/Oct"
- board text added: "BP"
- board text added: "FREQ"
- board text added: "FREQ ATTV"
- board text added: "HI"
- board text added: "IN 1"
- board text added: "IN 2"
- board text added: "LO"
- board text added: "MIX"
- board text added: "SLOPE"
- board text added: "SLOPE ATTV"
- board text added: "Serge VCFS rev 01"
- board text added: "This side towards panel"
- board text added: "VC FREQ"
- board text added: "VC SLOPE"
