File: serge-112-vcfq/serge-112-vcfq.kicad_pcb (KiCad board)
At the start: 2 copper layers, 0 parts

Commit message: Fixing issue with serge vcfq
Parts:
- added C1: 1nF, rumblesan-footprints:C_Rect_L7.0mm_W3.5mm_P5.00mm, F.Cu at (155.4, 144.4)
- added C10: 220pF, rumblesan-footprints:C_Axial_L12.0mm_D5.0mm_P15.00mm_Horizontal, F.Cu at (127.0, 79.2)
- added C11: 100nF, rumblesan-footprints:C_Rect_L7.0mm_W3.5mm_P5.00mm, F.Cu at (149.8, 79.2)
- added C12: 220pF, rumblesan-footprints:C_Axial_L12.0mm_D5.0mm_P15.00mm_Horizontal, F.Cu at (127.0, 61.7)
- added C13: 100nF, rumblesan-footprints:C_Rect_L7.0mm_W3.5mm_P5.00mm, F.Cu at (149.8, 61.7)
- added C14: 100nF, rumblesan-footprints:C_Rect_L7.0mm_W3.5mm_P5.00mm, F.Cu at (127.0, 170.2)
- added C15: 10uF, rumblesan-footprints:CP_Radial_D5.0mm_P2.50mm, F.Cu at (117.6, 34.8)
- added C16: 10uF, rumblesan-footprints:CP_Radial_D5.0mm_P2.50mm, F.Cu at (137.2, 35.6)
- added C17: 100nF, rumblesan-footprints:C_Rect_L7.0mm_W3.5mm_P5.00mm, F.Cu at (124.2, 42.7)
- added C18: 100nF, rumblesan-footprints:C_Rect_L7.0mm_W3.5mm_P5.00mm, F.Cu at (133.3, 42.7)
- added C2: 220pF, rumblesan-footprints:C_Rect_L7.0mm_W3.5mm_P5.00mm, F.Cu at (142.2, 157.3)
- added C3: 220pF, rumblesan-footprints:C_Rect_L7.0mm_W3.5mm_P5.00mm, F.Cu at (127.0, 178.1)
- added C4: 100nF, rumblesan-footprints:C_Rect_L7.0mm_W3.5mm_P5.00mm, F.Cu at (142.2, 165.1)
- added C5: 100nF, rumblesan-footprints:C_Rect_L7.0mm_W3.5mm_P5.00mm, F.Cu at (121.8, 105.7)
- added C6: 100nF, rumblesan-footprints:C_Rect_L7.0mm_W3.5mm_P5.00mm, F.Cu at (130.0, 120.7)
- added C7: 22pF, rumblesan-footprints:C_Rect_L7.0mm_W3.5mm_P5.00mm, F.Cu at (125.2, 102.4)
- added C8: 100nF, rumblesan-footprints:C_Rect_L7.0mm_W3.5mm_P5.00mm, F.Cu at (128.8, 114.8)
- added C9: 22pF, rumblesan-footprints:C_Rect_L7.0mm_W3.5mm_P5.00mm, F.Cu at (124.5, 69.8)
- added CX1: 33pF, rumblesan-footprints:C_Rect_L7.0mm_W3.5mm_P5.00mm, F.Cu at (144.0, 178.1)
- added CY1: 33pF, rumblesan-footprints:C_Rect_L7.0mm_W3.5mm_P5.00mm, F.Cu at (127.0, 156.5)
- added CZ1: 33pF, rumblesan-footprints:C_Rect_L7.0mm_W3.5mm_P5.00mm, F.Cu at (116.8, 120.9)
- added D1: 1n4148, rumblesan-footprints:Diode_THT_P7.62mm_Horizontal, F.Cu at (157.5, 158.5)
- added D2: 1n4148, rumblesan-footprints:Diode_THT_P7.62mm_Horizontal, F.Cu at (123.2, 170.4)
- added D3: 1n4148, rumblesan-footprints:Diode_THT_P7.62mm_Horizontal, F.Cu at (147.8, 178.6)
- added D4: 1n4148, rumblesan-footprints:Diode_THT_P7.62mm_Horizontal, F.Cu at (152.9, 113.0)
- added D5: 1n4148, rumblesan-footprints:Diode_THT_P7.62mm_Horizontal, F.Cu at (157.5, 125.5)
- added FREQ1: 50k Lin, rumblesan-footprints:Potentiometer_Alpha_RD901F-40-00D_Single_Vertical_CircularHoles, F.Cu at (97.8, 170.4)
- added GAIN1: 50k Lin, rumblesan-footprints:Potentiometer_Alpha_RD901F-40-00D_Single_Vertical_CircularHoles, F.Cu at (72.4, 170.4)
- added H1: MountingScrew_M3_Flathead, MountingHole:MountingHole_3.2mm_M3, F.Cu at (79.5, 42.7)
- added H2: MountingScrew_M3_Flathead, MountingHole:MountingHole_3.2mm_M3, F.Cu at (91.9, 141.0)
- added H3: MountingScrew_M3_Flathead, MountingHole:MountingHole_3.2mm_M3, F.Cu at (141.5, 42.7)
- added H4: MountingScrew_M3_Flathead, MountingHole:MountingHole_3.2mm_M3, F.Cu at (129.0, 141.0)
- added J1: Input_Header_Main, Connector_PinSocket_2.54mm:PinSocket_1x02_P2.54mm_Vertical, B.Cu at (157.5, 118.9)
- added J10: 1V/OCT, rumblesan-footprints:BananaJack_THT_JohnsonCinch_108-09, F.Cu at (97.8, 113.3)
- added J11: VC F, rumblesan-footprints:BananaJack_THT_JohnsonCinch_108-09, F.Cu at (97.8, 132.3)
- added J12: HIGH, rumblesan-footprints:BananaJack_THT_JohnsonCinch_108-09, F.Cu at (97.8, 37.1)
- added J13: POWER, rumblesan-footprints:Molex_KK-254_AE-6410-04A_1x04_P2.54mm_Vertical, F.Cu at (124.5, 35.3)
- added J14: BP, rumblesan-footprints:BananaJack_THT_JohnsonCinch_108-09, F.Cu at (72.4, 37.1)
- added J15: Conn_01x02_Female, Connector_PinSocket_2.54mm:PinSocket_1x02_P2.54mm_Vertical, B.Cu at (63.5, 66.8)
- added J16: Conn_01x02_Female, Connector_PinSocket_2.54mm:PinSocket_1x02_P2.54mm_Vertical, B.Cu at (87.9, 95.2)
- added J17: Range_Header_Main, Connector_PinSocket_2.54mm:PinSocket_1x04_P2.54mm_Vertical, B.Cu at (157.5, 82.0)
- added J18: Range_Header_IO, Connector_PinHeader_2.54mm:PinHeader_1x04_P2.54mm_Vertical, B.Cu at (63.5, 82.0)
- added J19: LOW, rumblesan-footprints:BananaJack_THT_JohnsonCinch_108-09, F.Cu at (97.8, 56.1)
- added J2: Input_Header_IO, Connector_PinHeader_2.54mm:PinHeader_1x02_P2.54mm_Vertical, B.Cu at (63.5, 118.9)
- added J20: Conn_01x02_Male, Connector_PinHeader_2.54mm:PinHeader_1x02_P2.54mm_Vertical, B.Cu at (157.5, 66.8)
- added J21: Conn_01x02_Male, Connector_PinHeader_2.54mm:PinHeader_1x02_P2.54mm_Vertical, B.Cu at (133.1, 95.2)
- added J22: Conn_01x02_Female, Connector_PinSocket_2.54mm:PinSocket_1x02_P2.54mm_Vertical, B.Cu at (82.0, 139.4)
- added J23: Conn_01x02_Male, Connector_PinHeader_2.54mm:PinHeader_1x02_P2.54mm_Vertical, B.Cu at (138.9, 139.4)
- added J24: Conn_01x06_Female, Connector_PinSocket_2.54mm:PinSocket_1x06_P2.54mm_Vertical, B.Cu at (106.7, 147.6)
- added J25: Conn_01x06_Male, Connector_PinHeader_2.54mm:PinHeader_1x06_P2.54mm_Vertical, B.Cu at (114.3, 147.6)
- added J3: VC Q, rumblesan-footprints:BananaJack_THT_JohnsonCinch_108-09, F.Cu at (72.4, 113.3)
- added J4: IN, rumblesan-footprints:BananaJack_THT_JohnsonCinch_108-09, F.Cu at (97.8, 75.2)
- added J5: AGC IN, rumblesan-footprints:BananaJack_THT_JohnsonCinch_108-09, F.Cu at (72.4, 75.2)
- added J6: TRIG, rumblesan-footprints:BananaJack_THT_JohnsonCinch_108-09, F.Cu at (97.8, 94.2)
- added J7: Input_Header_IO, Connector_PinHeader_2.54mm:PinHeader_1x02_P2.54mm_Vertical, B.Cu at (72.9, 162.6)
- added J8: NOTCH, rumblesan-footprints:BananaJack_THT_JohnsonCinch_108-09, F.Cu at (72.4, 56.1)
- added J9: Input_Header_Main, Connector_PinSocket_2.54mm:PinSocket_1x02_P2.54mm_Vertical, B.Cu at (148.1, 162.6)
- added Q1: 50k Lin, rumblesan-footprints:Potentiometer_Alpha_RD901F-40-00D_Single_Vertical_CircularHoles, F.Cu at (72.4, 151.4)
- added Q2: 50k Lin, rumblesan-footprints:Potentiometer_Alpha_RD901F-40-00D_Single_Vertical_CircularHoles, F.Cu at (72.4, 132.3)
- added R1: 110k, rumblesan-footprints:Resistor_THT_L6.3mm_D2.5mm_P10.16mm_Horizontal, F.Cu at (118.1, 165.6)
- added R10: 2k0, rumblesan-footprints:Resistor_THT_L6.3mm_D2.5mm_P10.16mm_Horizontal, F.Cu at (116.8, 178.1)
- added R11: 15k, rumblesan-footprints:Resistor_THT_L6.3mm_D2.5mm_P10.16mm_Horizontal, F.Cu at (119.9, 178.1)
- added R12: 100k, rumblesan-footprints:Resistor_THT_L6.3mm_D2.5mm_P10.16mm_Horizontal, F.Cu at (140.5, 177.5)
- added R13: 47k, rumblesan-footprints:Resistor_THT_L6.3mm_D2.5mm_P10.16mm_Horizontal, F.Cu at (150.9, 165.6)
- added R14: 100k, rumblesan-footprints:Resistor_THT_L6.3mm_D2.5mm_P10.16mm_Horizontal, F.Cu at (153.9, 175.8)
- added R15: 330R, rumblesan-footprints:Resistor_THT_L6.3mm_D2.5mm_P10.16mm_Horizontal, F.Cu at (123.2, 147.6)
- added R16: 15k, rumblesan-footprints:Resistor_THT_L6.3mm_D2.5mm_P10.16mm_Horizontal, F.Cu at (157.0, 175.8)
- added R17: 330R, rumblesan-footprints:Resistor_THT_L6.3mm_D2.5mm_P10.16mm_Horizontal, F.Cu at (154.2, 158.5)
- added R18: 330R, rumblesan-footprints:Resistor_THT_L6.3mm_D2.5mm_P10.16mm_Horizontal, F.Cu at (119.4, 95.2)
- added R19: 220k, rumblesan-footprints:Resistor_THT_L6.3mm_D2.5mm_P10.16mm_Horizontal, F.Cu at (152.9, 100.6)
- added R2: 100k, rumblesan-footprints:Resistor_THT_L6.3mm_D2.5mm_P10.16mm_Horizontal, F.Cu at (123.2, 150.6)
- added R20: 330k, rumblesan-footprints:Resistor_THT_L6.3mm_D2.5mm_P10.16mm_Horizontal, F.Cu at (151.1, 148.3)
- added R21: 330R, rumblesan-footprints:Resistor_THT_L6.3mm_D2.5mm_P10.16mm_Horizontal, F.Cu at (140.0, 100.6)
- added R22: 100k, rumblesan-footprints:Resistor_THT_L6.3mm_D2.5mm_P10.16mm_Horizontal, F.Cu at (150.1, 115.8)
- added R23: 47k, rumblesan-footprints:Resistor_THT_L6.3mm_D2.5mm_P10.16mm_Horizontal, F.Cu at (140.0, 118.9)
- added R24: 100k, rumblesan-footprints:Resistor_THT_L6.3mm_D2.5mm_P10.16mm_Horizontal, F.Cu at (140.0, 121.9)
- added R25: NotFitted, rumblesan-footprints:Resistor_THT_L6.3mm_D2.5mm_P10.16mm_Horizontal, F.Cu at (77.0, 124.5)
- added R26: 100k, rumblesan-footprints:Resistor_THT_L6.3mm_D2.5mm_P10.16mm_Horizontal, F.Cu at (140.0, 103.6)
- added R27: 100k, rumblesan-footprints:Resistor_THT_L6.3mm_D2.5mm_P10.16mm_Horizontal, F.Cu at (150.1, 112.8)
- added R28: 100k, rumblesan-footprints:Resistor_THT_L6.3mm_D2.5mm_P10.16mm_Horizontal, F.Cu at (150.1, 106.7)
- added R29: 47k, rumblesan-footprints:Resistor_THT_L6.3mm_D2.5mm_P10.16mm_Horizontal, F.Cu at (134.6, 98.8)
- added R3: 22k, rumblesan-footprints:Resistor_THT_L6.3mm_D2.5mm_P10.16mm_Horizontal, F.Cu at (133.3, 153.7)
- added R30: 100k, rumblesan-footprints:Resistor_THT_L6.3mm_D2.5mm_P10.16mm_Horizontal, F.Cu at (133.3, 115.6)
- added R31: 100k, rumblesan-footprints:Resistor_THT_L6.3mm_D2.5mm_P10.16mm_Horizontal, F.Cu at (140.0, 109.7)
- added R32: 1k, rumblesan-footprints:Resistor_THT_L6.3mm_D2.5mm_P10.16mm_Horizontal, F.Cu at (152.1, 139.4)
- added R33: 47k, rumblesan-footprints:Resistor_THT_L6.3mm_D2.5mm_P10.16mm_Horizontal, F.Cu at (134.6, 66.0)
- added R34: 330R, rumblesan-footprints:Resistor_THT_L6.3mm_D2.5mm_P10.16mm_Horizontal, F.Cu at (142.2, 69.6)
- added R35: 330R, rumblesan-footprints:Resistor_THT_L6.3mm_D2.5mm_P10.16mm_Horizontal, F.Cu at (142.2, 66.5)
- added R4: 47k, rumblesan-footprints:Resistor_THT_L6.3mm_D2.5mm_P10.16mm_Horizontal, F.Cu at (87.1, 150.9)
- added R5: 22k, rumblesan-footprints:Resistor_THT_L6.3mm_D2.5mm_P10.16mm_Horizontal, F.Cu at (123.2, 157.7)
- added R6: 47k, rumblesan-footprints:Resistor_THT_L6.3mm_D2.5mm_P10.16mm_Horizontal, F.Cu at (152.1, 142.5)
- added R7: 1M5, rumblesan-footprints:Resistor_THT_L6.3mm_D2.5mm_P10.16mm_Horizontal, F.Cu at (148.1, 148.3)
- added R8: 150k, rumblesan-footprints:Resistor_THT_L6.3mm_D2.5mm_P10.16mm_Horizontal, F.Cu at (142.0, 145.5)
- added R9: 100k, rumblesan-footprints:Resistor_THT_L6.3mm_D2.5mm_P10.16mm_Horizontal, F.Cu at (147.8, 165.6)
- added RV1: 100R, rumblesan-footprints:Potentiometer_THT_Bourns_3306P_Vertical, F.Cu at (120.4, 139.2)
- added SW1: SW_DPST_x2, rumblesan-footprints:SW_NKK_M2021SS1W03, F.Cu at (72.4, 94.2)
- added U1: TL074, rumblesan-footprints:DIP-14_W7.62mm_Socket, F.Cu at (130.8, 159.0)
- added U2: TL072, rumblesan-footprints:DIP-8_W7.62mm_Socket, F.Cu at (116.8, 117.1)
- added VCA1: CGS108, rumblesan-footprints:Serge_GainCell_Vertical, F.Cu at (116.8, 126.2)
- added VCA2: CGS108, rumblesan-footprints:Serge_GainCell_Vertical, F.Cu at (116.8, 84.6)
- added VCA3: CGS108, rumblesan-footprints:Serge_GainCell_Vertical, F.Cu at (116.8, 48.8)
- added VCF1: 50k Lin, rumblesan-footprints:Potentiometer_Alpha_RD901F-40-00D_Single_Vertical_CircularHoles, F.Cu at (97.8, 151.4)
- added mouse-bite-2.54mm-slot: VAL**, rumblesan-footprints:mouse-bite-2.54mm-slot, F.Cu at (110.5, 167.9)
- added mouse-bite-2.54mm-slot: VAL**, rumblesan-footprints:mouse-bite-2.54mm-slot, F.Cu at (110.5, 131.1)
- added mouse-bite-2.54mm-slot: VAL**, rumblesan-footprints:mouse-bite-2.54mm-slot, F.Cu at (110.5, 101.9)
- added mouse-bite-2.54mm-slot: VAL**, rumblesan-footprints:mouse-bite-2.54mm-slot, F.Cu at (110.5, 77.5)
- added mouse-bite-2.54mm-slot: VAL**, rumblesan-footprints:mouse-bite-2.54mm-slot, F.Cu at (110.5, 46.0)
Routing:
- net +12V: track 0.00 -> 180.8 mm
- net -12V: track 0.00 -> 164.9 mm
- net Net-(GAIN1-Pad3): track 0.00 -> 116.5 mm
- net FREQ-CONTROL: track 0.00 -> 112.7 mm
- net /RANGE2_HI_MAIN: track 0.00 -> 108.9 mm
- net /RANGE1_HI_MAIN: track 0.00 -> 75.6 mm
- net /HIGH_IO: track 0.00 -> 70.2 mm
- net /IN_IO: track 0.00 -> 67.3 mm
- net +12VA: track 0.00 -> 62.5 mm
- net /TRIG_IO: track 0.00 -> 56.0 mm
- net /AGC_IO: track 0.00 -> 55.9 mm
- net Net-(R16-Pad2): track 0.00 -> 49.7 mm
- net /NOTCH_IO: track 0.00 -> 48.8 mm
- net Net-(CZ1-Pad2): track 0.00 -> 46.2 mm
- net /1VOCT_IO: track 0.00 -> 46.0 mm
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- added copper zone on B.Cu, net GNDA
- added copper zone on F.Cu, net GNDA
- added copper zone on B.Cu, net GNDREF
- added copper zone on F.Cu, net GNDREF
Other:
- board outline added: 99.1 x 150.6 mm
- rule pad_to_mask_clearance: 0.0508 -> 0
- board text added: "+V"
- board text added: "-V"
- board text added: "1V/OCT"
- board text added: "AGC IN"
- board text added: "BP"
- board text added: "HIGH"
- board text added: "IN"
- board text added: "LOW"
- board text added: "NOTCH"
- board text added: "RANGE"
- board text added: "Serge VCFQ rev 1.0"
- board text added: "TRIG"
- board text added: "This side toward panel"
- board text added: "VC F"
- board text added: "VC Q"
- board text added: "VC Q ATTN"
