File: serge-r6-gate-ringmod/serge-r6-gate-ringmod.sch (KiCad schematic (older format))
At the start: 59 parts, among them J1 LOG_CV/VC_X, J10 LIN_CV_Y_IN_SEL, J11 DC_IN_VC_Y_SEL, J2 AC_INPUT/INPUT_X, J3 DC_INPUT/Y_IN, J4 LIN_CV_INPUT_Y_SEL, J5 LIN_CV/VC_Y, J6 OUT, J7 CTRL_HEADER, J8 MAIN_HEADER, J9 Conn_01x04_Male, Q1 2N3906, Q2 2N3906, Q3 2N3906, U1 CA3080, U2 TL071

Commit message: Updating serge r6 gate
Parts:
- removed U2: TL071, Package_DIP:DIP-8_W7.62mm_Socket, symbol Amplifier_Operational:TL071
- added U?: LM301, symbol Amplifier_Operational:LM301
- C3: value 220pf -> 47pf
- RV1, RV2, RV3: value 25k -> 20k
Connections:
- net +12V: now also U?.7 (V+)
- net -12V: now also U?.4 (V-)
- net at C3.2, R21.2, U1.6: now also U?.2 (-)
- net at JP1.2, R18.1: now also U?.3 (+)
- net at C3.1, R21.1, R22.2: now also U?.6
Changed lines of the file:
@@
 $EndDescr
-$Comp
-L Amplifier_Operational:CA3080 U1
-U 1 1 61740BAF
-P 4200 5750
-F 0 "U1" H 4544 5796 50  0000 L CNN
-F 1 "CA3080" H 4544 5705 50  0000 L CNN
-F 2 "Package_DIP:DIP-8_W7.62mm_Socket" H 4200 5750 50  0001 C CNN
-F 3 "http://www.intersil.com/content/dam/Intersil/documents/ca30/ca3080-a.pdf" H 4200 5850 50  0001 C CNN
-	1    4200 5750
-	1    0    0    -1
-$EndComp
 $Comp
 L Transistor_BJT:2N3906 Q3
@@
 $EndComp
 $Comp
-L Amplifier_Operational:TL071 U2
-U 1 1 617444C5
-P 5450 5850
-F 0 "U2" H 5650 5550 50  0000 L CNN
-F 1 "TL071" H 5650 5450 50  0000 L CNN
-F 2 "Package_DIP:DIP-8_W7.62mm_Socket" H 5500 5900 50  0001 C CNN
-F 3 "http://www.ti.com/lit/ds/symlink/tl071.pdf" H 5600 6000 50  0001 C CNN
-	1    5450 5850
-	1    0    0    1
-$EndComp
-$Comp
 L BananaJacks:BananaJack_PanelMount J2
 U 1 1 61746101
@@
 P 1650 4700
 F 0 "RV1" H 1580 4746 50  0000 R CNN
-F 1 "25k" H 1580 4655 50  0000 R CNN
+F 1 "20k" H 1580 4655 50  0000 R CNN
 F 2 "rumblesan-footprints:Potentiometer_THT_Bourns_3306P_Vertical" H 1650 4700 50  0001 C CNN
 F 3 "~" H 1650 4700 50  0001 C CNN
 	1    1650 4700
-	1    0    0    -1
-$EndComp
-$Comp
-L power:GND #PWR012
-U 1 1 6174CBA8
-P 3900 3850
-F 0 "#PWR012" H 3900 3600 50  0001 C CNN
-F 1 "GND" H 3905 3677 50  0000 C CNN
-F 2 "" H 3900 3850 50  0001 C CNN
-F 3 "" H 3900 3850 50  0001 C CNN
-	1    3900 3850
 	1    0    0    -1
 $EndComp
@@
 	3600 7000 3600 6900
 Wire Wire Line
-	3750 5250 3750 5650
-Wire Wire Line
-	3750 5650 3900 5650
-Connection ~ 3200 5250
-Wire Wire Line
 	3600 6450 3750 6450
 Wire Wire Line
@@
 Wire Wire Line
 	4200 3300 4200 3350
-Wire Wire Line
-	3900 3750 3900 3850
 $Comp
 L Device:R R6
@@
 P 1850 3550
 F 0 "RV2" H 1780 3596 50  0000 R CNN
-F 1 "25k" H 1780 3505 50  0000 R CNN
+F 1 "20k" H 1780 3505 50  0000 R CNN
 F 2 "rumblesan-footprints:Potentiometer_THT_Bourns_3306P_Vertical" H 1850 3550 50  0001 C CNN
 F 3 "~" H 1850 3550 50  0001 C CNN
@@
 	2650 2950 2650 3550
 $Comp
-L Device:R R15
-U 1 1 61770154
-P 4200 4100
-F 0 "R15" H 4270 4146 50  0000 L CNN
-F 1 "15k" H 4270 4055 50  0000 L CNN
-F 2 "rumblesan-footprints:Resistor_THT_L6.3mm_D2.5mm_P10.16mm_Horizontal" V 4130 4100 50  0001 C CNN
-F 3 "~" H 4200 4100 50  0001 C CNN
-	1    4200 4100
-	1    0    0    -1
-$EndComp
-Wire Wire Line
-	4200 3750 4200 3950
-$Comp
 L Device:R R17
 U 1 1 617719DF
@@
 Wire Wire Line
 	6350 3500 6350 3600
-Wire Wire Line
-	3200 5250 3750 5250
-Wire Wire Line
-	3750 4700 3750 5250
-Wire Wire Line
-	2250 4700 3750 4700
-Connection ~ 3750 5250
 $Comp
 L Device:R R10
@@
 $EndComp
 Wire Wire Line
-	4200 4250 4200 5450
-Wire Wire Line
 	2650 3550 3600 3550
 Wire Wire Line
@@
 P 4050 1100
 F 0 "RV3" V 3843 1100 50  0000 C CNN
-F 1 "25k" V 3934 1100 50  0000 C CNN
+F 1 "20k" V 3934 1100 50  0000 C CNN
 F 2 "rumblesan-footprints:Potentiometer_THT_Bourns_3306P_Vertical" H 4050 1100 50  0001 C CNN
 F 3 "~" H 4050 1100 50  0001 C CNN
@@
 P 5400 4500
 F 0 "C3" V 5148 4500 50  0000 C CNN
-F 1 "220pf" V 5239 4500 50  0000 C CNN
+F 1 "47pf" V 5239 4500 50  0000 C CNN
 F 2 "Capacitor_THT:C_Rect_L7.0mm_W2.5mm_P5.00mm" H 5438 4350 50  0001 C CNN
 F 3 "~" H 5400 4500 50  0001 C CNN
@@
 Wire Wire Line
 	4100 6050 4100 6200
-$Comp
-L power:+12V #PWR013
-U 1 1 617E69EB
-P 4000 5250
-F 0 "#PWR013" H 4000 5100 50  0001 C CNN
-F 1 "+12V" H 4015 5423 50  0000 C CNN
-F 2 "" H 4000 5250 50  0001 C CNN
-F 3 "" H 4000 5250 50  0001 C CNN
-	1    4000 5250
-	1    0    0    -1
-$EndComp
-Wire Wire Line
-	4000 5250 4000 5350
-Wire Wire Line
-	4000 5350 4100 5350
-Wire Wire Line
-	4100 5350 4100 5450
 $Comp
 L Device:Jumper_NO_Small JP1
@@
 Text Notes 3300 7600 0    50   ~ 0
 Bridge for RingMod
+$Comp
+L Amplifier_Operational:LM301 U?
+U 1 1 60FC436F
+P 5450 5850
+F 0 "U?" H 5794 5804 50  0000 L CNN
+F 1 "LM301" H 5794 5895 50  0000 L CNN
+F 2 "" H 5500 5900 50  0001 C CNN
+F 3 "http://www.ti.com/lit/ds/symlink/lm101a-n.pdf" H 5500 6000 50  0001 C CNN
+	1    5450 5850
+	1    0    0    1
+$EndComp
+Connection ~ 3200 5250
+Wire Wire Line
+	3750 5650 3900 5650
+Wire Wire Line
+	4100 5350 4100 5450
+Wire Wire Line
+	4000 5350 4100 5350
+Wire Wire Line
+	4000 5250 4000 5350
+$Comp
+L power:+12V #PWR013
+U 1 1 617E69EB
+P 4000 5250
+F 0 "#PWR013" H 4000 5100 50  0001 C CNN
+F 1 "+12V" H 4015 5423 50  0000 C CNN
+F 2 "" H 4000 5250 50  0001 C CNN
+F 3 "" H 4000 5250 50  0001 C CNN
+	1    4000 5250
+	1    0    0    -1
+$EndComp
+Wire Wire Line
+	4200 4250 4200 5450
+Connection ~ 3750 5250
+Wire Wire Line
+	2250 4700 3750 4700
+Wire Wire Line
+	3750 4700 3750 5250
+Wire Wire Line
+	3200 5250 3750 5250
+Wire Wire Line
+	4200 3750 4200 3950
+$Comp
+L Device:R R15
+U 1 1 61770154
+P 4200 4100
+F 0 "R15" H 4270 4146 50  0000 L CNN
+F 1 "15k" H 4270 4055 50  0000 L CNN
+F 2 "rumblesan-footprints:Resistor_THT_L6.3mm_D2.5mm_P10.16mm_Horizontal" V 4130 4100 50  0001 C CNN
+F 3 "~" H 4200 4100 50  0001 C CNN
+	1    4200 4100
+	1    0    0    -1
+$EndComp
+Wire Wire Line
+	3900 3750 3900 3850
+Wire Wire Line
+	3750 5250 3750 5650
+$Comp
+L power:GND #PWR012
+U 1 1 6174CBA8
+P 3900 3850
+F 0 "#PWR012" H 3900 3600 50  0001 C CNN
+F 1 "GND" H 3905 3677 50  0000 C CNN
+F 2 "" H 3900 3850 50  0001 C CNN
+F 3 "" H 3900 3850 50  0001 C CNN
+	1    3900 3850
+	1    0    0    -1
+$EndComp
+$Comp
+L Amplifier_Operational:CA3080 U1
+U 1 1 61740BAF
+P 4200 5750
+F 0 "U1" H 4544 5796 50  0000 L CNN
+F 1 "CA3080" H 4544 5705 50  0000 L CNN
+F 2 "Package_DIP:DIP-8_W7.62mm_Socket" H 4200 5750 50  0001 C CNN
+F 3 "http://www.intersil.com/content/dam/Intersil/documents/ca30/ca3080-a.pdf" H 4200 5850 50  0001 C CNN
+	1    4200 5750
+	1    0    0    -1
+$EndComp
 $EndSCHEMATC
