File: dual-digi-delay/dual-digi-delay.kicad_pcb (KiCad board)
At the start: 2 copper layers, 148.8 x 152.9 mm, 198 parts, among them J1 TopBoardPowerRecv, J10 Delay Time Control, J11 Delay1 CV, J12 Delay2 CV, J13 Delay Send Return, J14 LowerBoardPowerSend, J15 Main Power, J16 Feedback Audio, J17 Delay Wet, J18 Delay1 CV, J19 Delay2 CV, J2 Delay Audio, J20 MidBoardPowerSend, J21 Delay Time Control, J22 Delay Audio, J23 Delay Out, J24 Output Audio, J25 DELAY2_CV, J26 DELAY1_CV, J27 AUDIO_IN, J28 MIX_OUT, J29 DELAY1_WET_OUT, J3 Input Audio, J30 DELAY2_WET_OUT, J31 Feedback Audio, J4 Output Audio, J5 Delay Out, J6 Delay Wet, J7 Input Audio, J8 Delay Send Return, J9 MidBoardPowerRecv, Q1 2N3904, Q2 2N3904, Q3 2N3904, Q4 2N3904, Q5 2N3904, Q6 2N3904, SW1 CV_JOIN, SW2 Delay 2 Input, U1 TL072, U2 TL072, U3 PT2399, U4 PT2399, U5 TL074, U6 TL074, U7 LM7805_TO220, U8 TL072

Commit message: Final revision of dual digi delay
Parts:
- removed H7, H8, H9: MountingHole, MountingHole:MountingHole_3.2mm_M3_ISO7380_Pad
- removed J17: Delay Wet, Connector_PinSocket_2.54mm:PinSocket_1x02_P2.54mm_Vertical
- removed J18: Delay1 CV, Connector_PinSocket_2.54mm:PinSocket_1x04_P2.54mm_Vertical
- removed J19: Delay2 CV, Connector_PinSocket_2.54mm:PinSocket_1x06_P2.54mm_Vertical
- removed J22: Delay Audio, Connector_PinSocket_2.54mm:PinSocket_1x04_P2.54mm_Vertical
- removed JP1, JP2: Jumper_3_Bridged12, Jumper:SolderJumper-3_P1.3mm_Bridged12_RoundedPad1.0x1.5mm_NumberLabels
- removed R60, R61: 47k, rumblesan-footprints:Resistor_THT_L6.3mm_D2.5mm_P10.16mm_Horizontal
- added C56: 10pF, rumblesan-footprints:C_Rect_L7.0mm_W3.5mm_P5.00mm, F.Cu at (110.2, 161.3)
- added D13: 1n4148, rumblesan-footprints:Diode_THT_P7.62mm_Horizontal, F.Cu at (86.9, 171.2)
- added D14: 1n4148, rumblesan-footprints:Diode_THT_P7.62mm_Horizontal, F.Cu at (79.2, 174.5)
- added D15: 1n4148, rumblesan-footprints:Diode_THT_P7.62mm_Horizontal, F.Cu at (107.7, 171.2)
- added D16: 1n4148, rumblesan-footprints:Diode_THT_P7.62mm_Horizontal, F.Cu at (115.3, 174.5)
- added J32: Delay Send, Connector_PinSocket_2.54mm:PinSocket_1x02_P2.54mm_Vertical, F.Cu at (169.4, 98.0)
- added J33: Delay Return, Connector_PinSocket_2.54mm:PinSocket_1x02_P2.54mm_Vertical, F.Cu at (169.4, 69.8)
- added J38: Delay2_CV, Connector_PinHeader_2.54mm:PinHeader_1x06_P2.54mm_Vertical, B.Cu at (68.8, 148.6)
- added J39: Delay2_CV, Connector_PinSocket_2.54mm:PinSocket_1x06_P2.54mm_Vertical, F.Cu at (119.1, 148.6)
- added R64: 10k, rumblesan-footprints:Resistor_THT_L6.3mm_D2.5mm_P10.16mm_Horizontal, F.Cu at (76.2, 167.6)
- added R65: 1k, rumblesan-footprints:Resistor_THT_L6.3mm_D2.5mm_P10.16mm_Horizontal, F.Cu at (89.4, 177.8)
- added R66: 10k, rumblesan-footprints:Resistor_THT_L6.3mm_D2.5mm_P10.16mm_Horizontal, F.Cu at (118.4, 167.6)
- added R67: 1k, rumblesan-footprints:Resistor_THT_L6.3mm_D2.5mm_P10.16mm_Horizontal, F.Cu at (105.2, 177.8)
- added R68: 47k, rumblesan-footprints:Resistor_THT_L6.3mm_D2.5mm_P10.16mm_Horizontal, F.Cu at (105.2, 147.6)
- added R69: 47k, rumblesan-footprints:Resistor_THT_L6.3mm_D2.5mm_P10.16mm_Horizontal, F.Cu at (89.4, 147.6)
- added mouse-bite-2mm-slot: VAL**, Panelization:mouse-bite-2mm-slot, F.Cu at (72.1, 40.6)
- added mouse-bite-2mm-slot: VAL**, Panelization:mouse-bite-2mm-slot, F.Cu at (72.1, 66.0)
- added mouse-bite-2mm-slot: VAL**, Panelization:mouse-bite-2mm-slot, F.Cu at (122.4, 40.6)
- added mouse-bite-2mm-slot: VAL**, Panelization:mouse-bite-2mm-slot, F.Cu at (122.4, 66.0)
- added mouse-bite-2mm-slot: VAL**, Panelization:mouse-bite-2mm-slot, F.Cu at (72.1, 167.6)
- added mouse-bite-2mm-slot: VAL**, Panelization:mouse-bite-2mm-slot, F.Cu at (122.4, 167.6)
- added mouse-bite-2mm-slot: VAL**, Panelization:mouse-bite-2mm-slot, F.Cu at (72.1, 142.5)
- added mouse-bite-2mm-slot: VAL**, Panelization:mouse-bite-2mm-slot, F.Cu at (122.4, 142.2)
- added mouse-bite-2mm-slot: VAL**, Panelization:mouse-bite-2mm-slot, F.Cu at (72.1, 116.8)
- added mouse-bite-2mm-slot: VAL**, Panelization:mouse-bite-2mm-slot, F.Cu at (122.4, 116.8)
- added mouse-bite-2mm-slot: VAL**, Panelization:mouse-bite-2mm-slot, F.Cu at (122.4, 91.4)
- added mouse-bite-2mm-slot: VAL**, Panelization:mouse-bite-2mm-slot, F.Cu at (72.1, 91.4)
- H1, H2, H3, H4, H5, H6: value MountingHole -> MountingHole_Pad; footprint MountingHole:MountingHole_3.2mm_M3_ISO7380_Pad -> MountingHole:MountingHole_3.2mm_M3_Pad
- J11: value Delay1 CV -> Delay1_CV; footprint Connector_PinHeader_2.54mm:PinHeader_1x04_P2.54mm_Vertical -> Connector_PinHeader_2.54mm:PinHeader_1x06_P2.54mm_Vertical
- J12: value Delay2 CV -> Delay1_CV; footprint Connector_PinHeader_2.54mm:PinHeader_1x06_P2.54mm_Vertical -> Connector_PinSocket_2.54mm:PinSocket_1x06_P2.54mm_Vertical; moved to F.Cu
- J13: value Delay Send Return -> Delay Send; footprint Connector_PinSocket_2.54mm:PinSocket_1x04_P2.54mm_Vertical -> Connector_PinHeader_2.54mm:PinHeader_1x02_P2.54mm_Vertical; moved to B.Cu
- J2: value Delay Audio -> DelayAudio; footprint Connector_PinHeader_2.54mm:PinHeader_1x04_P2.54mm_Vertical -> Connector_PinHeader_2.54mm:PinHeader_1x06_P2.54mm_Vertical
- J6: value Delay Wet -> DelayAudio; footprint Connector_PinHeader_2.54mm:PinHeader_1x02_P2.54mm_Vertical -> Connector_PinSocket_2.54mm:PinSocket_1x06_P2.54mm_Vertical; moved to F.Cu
- J8: value Delay Send Return -> Delay Return; footprint Connector_PinHeader_2.54mm:PinHeader_1x04_P2.54mm_Vertical -> Connector_PinHeader_2.54mm:PinHeader_1x02_P2.54mm_Vertical
- R35: value 47k -> 100k
- moved H4 147.0 mm to (97.3, 177.0)
- moved H5 95.2 mm to (127.3, 31.8)
- moved J6 77.6 mm to (119.1, 75.9)
- moved R32 62.1 mm to (115.3, 167.9), turned to 180 degrees
- moved J12 61.5 mm to (75.4, 148.6), turned to 0 degrees
- moved R53 60.1 mm to (79.8, 114.3), turned to 0 degrees
- moved Q4 58.2 mm to (77.0, 110.0), turned to 0 degrees
- moved R31 57.1 mm to (115.3, 164.8), turned to 180 degrees
- moved R52 56.1 mm to (95.8, 104.9), turned to 180 degrees
- moved R38 54.8 mm to (105.2, 154.7)
- moved H2 54.6 mm to (47.0, 177.0)
- moved H1 52.7 mm to (26.7, 31.8)
- moved H3 52.7 mm to (77.0, 31.8)
- moved R43 51.4 mm to (115.3, 141.5)
- moved J13 50.2 mm to (119.1, 98.0), turned to 0 degrees
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Connections:
- C40 pad 1: Net-(C40-Pad1) -> /CVControl/DELAY1_CV_CTRL
- DELAY1_CV_ATTV1 pad 3: /CVInputs/DELAY1_CV_INPUT -> /CVInputs/DELAY1_CV_CTRL
- DELAY1_TIME1 pad 3: Net-(DELAY1_TIME1-Pad3) -> /TOP_0V
- DELAY2_TIME1 pad 3: Net-(DELAY2_TIME1-Pad3) -> /TOP_0V
- H1 pad 1: (no net) -> /TOP_0V
- H2 pad 1: (no net) -> /TOP_0V
- H3 pad 1: (no net) -> /MID_0V
- H4 pad 1: (no net) -> /MID_0V
- H5 pad 1: (no net) -> GND
- H6 pad 1: (no net) -> GND
- J1 pad 1: /CVInputs/+V -> /TOP_0V
- J11 pad 1: /CVInputs/DELAY1_CV_ATTV -> /CVInputs/JOIN_CV_SOURCE
- J11 pad 2: /CVInputs/DELAY1_CV_INPUT -> /CVInputs/DELAY1_CONTROL
- J11 pad 3: /CVInputs/DELAY1_CONTROL -> /CVInputs/DELAY1_CV_ATTV
- J11 pad 4: /CVInputs/JOIN_CV_SOURCE -> /CVInputs/DELAY1_CV_CTRL
- J12 pad 1: /CVInputs/DELAY2_CV_ATTV -> /CVControl/DELAY1_CV_JOIN_OUT
- J12 pad 2: /CVInputs/DELAY2_CV_CTRL -> /CVControl/DELAY1_CONTROL
- J12 pad 3: /CVInputs/DELAY2_CV_INPUT -> /CVControl/DELAY1_CV_ATTV
- J12 pad 4: /CVInputs/JOIN_CV -> /CVControl/DELAY1_CV_CTRL
- J12 pad 5: /CVInputs/DELAY2_CONTROL -> /CVControl/DELAY1_CV_INPUT
- J12 pad 6: /TOP_0V -> /MID_0V
- J13 pad 1: /PT2399-Delay-1/AUDIO_IN -> /InputMix/INPUT_MIX
- J13 pad 2: /PT2399-Delay-1/AUDIO_OUT -> Net-(J13-Pad2)
- J2 pad 2: /AudioIO/INPUT_MIX -> /AudioIO/DELAY1_WET_LEVEL
- J2 pad 3: /AudioIO/DELAY2_SOURCE -> /AudioIO/DELAY2_WET_LEVEL
- J20 pad 1: /MID_+V -> /MID_0V
- J6 pad 1: /AudioIO/DELAY1_WET_LEVEL -> /DelayOut/DELAY1_WET
- J6 pad 2: /AudioIO/DELAY2_WET_LEVEL -> /OutputMix/DELAY1_WET_LEVEL
- J8 pad 1: /InputMix/INPUT_MIX -> /DelayOut/DELAY1_WET
- J8 pad 2: /DelayOut/DELAY1_WET -> /DelayOut/DELAY2_WET
- R1 pad 2: /OutputMix/DELAY2_WET -> /OutputMix/DELAY2_WET_LEVEL
- R2 pad 2: /OutputMix/DELAY1_WET -> /OutputMix/DELAY1_WET_LEVEL
- R31 pad 2: Net-(R31-Pad2) -> Net-(C56-Pad2)
- R32 pad 2: Net-(R31-Pad2) -> Net-(C56-Pad2)
- R33 pad 1: Net-(R31-Pad2) -> Net-(C56-Pad2)
- R34 pad 1: Net-(C40-Pad1) -> /CVControl/DELAY1_CV_CTRL
- R35 pad 2: Net-(C40-Pad1) -> /CVControl/DELAY1_CV_CTRL
- R37 pad 1: Net-(C42-Pad2) -> /CVControl/DELAY1_CONTROL
- R37 pad 2: /CVControl/DELAY1_CONTROL -> Net-(C42-Pad2)
- R39 pad 1: Net-(C42-Pad2) -> Net-(C44-Pad2)
- R43 pad 1: Net-(C43-Pad2) -> /CVControl/DELAY2_CONTROL
- R43 pad 2: /CVControl/DELAY2_CONTROL -> Net-(C41-Pad2)
- R62 pad 1: /DelayOut/DELAY1_WET_OUT -> /DelayOut/DELAY2_WET_OUT
- R63 pad 1: /DelayOut/DELAY2_WET_OUT -> /DelayOut/DELAY1_WET_OUT
- U5 pad 1: Net-(C41-Pad1) -> Net-(C46-Pad2)
- U5 pad 13: Net-(C43-Pad2) -> Net-(C45-Pad1)
- U5 pad 14: Net-(C43-Pad1) -> Net-(C45-Pad2)
- U5 pad 2: Net-(C41-Pad2) -> Net-(C46-Pad1)
- U5 pad 3: /CVControl/DELAY2_CV_ATTV -> /MID_0V
- U5 pad 6: Net-(R31-Pad2) -> Net-(C44-Pad2)
- U5 pad 7: /CVControl/DELAY2_CV_CTRL -> Net-(C44-Pad1)
- U5 pad 8: Net-(C45-Pad2) -> Net-(C43-Pad1)
- U5 pad 9: Net-(C45-Pad1) -> Net-(C43-Pad2)
- U6 pad 12: /MID_0V -> /CVControl/DELAY2_CV_ATTV
- U6 pad 13: Net-(C44-Pad2) -> Net-(C41-Pad2)
- U6 pad 14: Net-(C44-Pad1) -> Net-(C41-Pad1)
- U6 pad 3: /MID_0V -> /CVControl/DELAY1_CV_ATTV
- U6 pad 5: /CVControl/DELAY1_CV_ATTV -> /MID_0V
- U6 pad 7: Net-(C40-Pad1) -> /CVControl/DELAY1_CV_CTRL
- U6 pad 8: Net-(C46-Pad2) -> /CVControl/DELAY2_CV_CTRL
- U6 pad 9: Net-(C46-Pad1) -> Net-(C56-Pad2)
- U8 pad 3: /DelayOut/DELAY2_WET -> /DelayOut/DELAY1_WET
- U8 pad 5: /DelayOut/DELAY1_WET -> /DelayOut/DELAY2_WET
Routing:
- net GND: track 4.04 -> 103.9 mm, vias 0 -> 12
- net /AudioIO/DRY_AUDIO_LEVEL: track 0.00 -> 96.3 mm, vias 0 -> 2
- net /AudioIO/DRY_AUDIO_INPUT: track 0.00 -> 63.7 mm
- net /CVControl/DELAY1_CV_CTRL: track 0.00 -> 46.7 mm
- net /AudioIO/DELAY2_SOURCE: track 0.00 -> 45.8 mm
- net /AudioIO/DELAY1_WET: track 0.00 -> 44.7 mm
- net /DelayOut/DELAY2_WET: track 4.06 -> 43.8 mm
- net /PT2399-Delay-2/DELAY_TIME_CTRL: track 65.7 -> 27.8 mm
- net /CVControl/DELAY2_CONTROL: track 46.3 -> 8.69 mm
- net /AudioIO/INPUT_MIX: track 0.00 -> 36.7 mm
- net /CVInputs/JOIN_CV: track 0.00 -> 36.2 mm
- net /OutputMix/DELAY_MIX: track 0.00 -> 35.6 mm
- net Net-(D1-Pad2): track 0.00 -> 35.0 mm
- net /CVInputs/DELAY2_CONTROL: track 0.00 -> 35.0 mm
- net /CVInputs/DELAY1_CV_INPUT: track 0.00 -> 34.7 mm
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- added copper zone on B.Cu, net /MID_0V
- added copper zone on F.Cu, net /MID_0V
- added copper zone on B.Cu, net /TOP_0V
- added copper zone on F.Cu, net /TOP_0V
- added copper zone on B.Cu, net GND
- added copper zone on F.Cu, net GND
Other:
- outline, holes or cut-outs redrawn
- board text added: "+V"
- board text added: "-V"
- board text added: "DELAY1 CV"
- board text added: "DELAY1 WET"
- board text added: "DELAY2 CV"
- board text added: "DELAY2 WET"
- board text added: "Dual PT2399 Digi Delay Revision 01"
- board text added: "Guy John <guy@rumblesan.com>"
- board text added: "INPUT"
- board text added: "JOIN"
- board text added: "MAIN OUT"
- board text added: "SERIES/PARALLEL"
- board text added: "THIS SIDE TOWARDS PANEL"
