File: dual-digi-delay/dual-digi-delay.sch (KiCad schematic (older format))
At the start: 35 parts, among them J1 TopBoardPowerRecv, J10 Delay Time Control, J11 Delay1 CV, J12 Delay2 CV, J13 Delay Send Return, J14 LowerBoardPowerSend, J15 Main Power, J16 Feedback Audio, J17 Delay Wet, J18 Delay1 CV, J19 Delay2 CV, J2 Delay Audio, J20 MidBoardPowerSend, J21 Delay Time Control, J22 Delay Audio, J23 Delay Out, J24 Output Audio, J3 Input Audio, J31 Feedback Audio, J4 Output Audio, J5 Delay Out, J6 Delay Wet, J7 Input Audio, J8 Delay Send Return, J9 MidBoardPowerRecv

Commit message: Final revision of dual digi delay
Parts:
- removed H1, H2, H3, H4, H5, H6, H7, H8, H9: MountingHole, MountingHole:MountingHole_3.2mm_M3_ISO7380_Pad, symbol Mechanical:MountingHole
- removed J11: Delay1 CV, Connector_PinHeader_2.54mm:PinHeader_1x04_P2.54mm_Vertical, symbol Connector:Conn_01x04_Male
- removed J12: Delay2 CV, Connector_PinHeader_2.54mm:PinHeader_1x06_P2.54mm_Vertical, symbol Connector:Conn_01x06_Male
- removed J13: Delay Send Return, Connector_PinSocket_2.54mm:PinSocket_1x04_P2.54mm_Vertical, symbol Connector:Conn_01x04_Female
- removed J17: Delay Wet, Connector_PinSocket_2.54mm:PinSocket_1x02_P2.54mm_Vertical, symbol Connector:Conn_01x02_Female
- removed J18: Delay1 CV, Connector_PinSocket_2.54mm:PinSocket_1x04_P2.54mm_Vertical, symbol Connector:Conn_01x04_Female
- removed J19: Delay2 CV, Connector_PinSocket_2.54mm:PinSocket_1x06_P2.54mm_Vertical, symbol Connector:Conn_01x06_Female
- removed J2: Delay Audio, Connector_PinHeader_2.54mm:PinHeader_1x04_P2.54mm_Vertical, symbol Connector:Conn_01x04_Male
- removed J22: Delay Audio, Connector_PinSocket_2.54mm:PinSocket_1x04_P2.54mm_Vertical, symbol Connector:Conn_01x04_Female
- removed J6: Delay Wet, Connector_PinHeader_2.54mm:PinHeader_1x02_P2.54mm_Vertical, symbol Connector:Conn_01x02_Male
- removed J8: Delay Send Return, Connector_PinHeader_2.54mm:PinHeader_1x04_P2.54mm_Vertical, symbol Connector:Conn_01x04_Male
- added H1, H2, H3, H4, H5, H6: MountingHole_Pad, MountingHole:MountingHole_3.2mm_M3_Pad, symbol Mechanical:MountingHole_Pad
- added J11: Delay1_CV, Connector_PinHeader_2.54mm:PinHeader_1x06_P2.54mm_Vertical, symbol Connector:Conn_01x06_Male
- added J12: Delay1_CV, Connector_PinSocket_2.54mm:PinSocket_1x06_P2.54mm_Vertical, symbol Connector:Conn_01x06_Female
- added J13: Delay Send, Connector_PinHeader_2.54mm:PinHeader_1x02_P2.54mm_Vertical, symbol Connector:Conn_01x02_Male
- added J2: DelayAudio, Connector_PinHeader_2.54mm:PinHeader_1x06_P2.54mm_Vertical, symbol Connector:Conn_01x06_Male
- added J32: Delay Send, Connector_PinSocket_2.54mm:PinSocket_1x02_P2.54mm_Vertical, symbol Connector:Conn_01x02_Female
- added J33: Delay Return, Connector_PinSocket_2.54mm:PinSocket_1x02_P2.54mm_Vertical, symbol Connector:Conn_01x02_Female
- added J38: Delay2_CV, Connector_PinHeader_2.54mm:PinHeader_1x06_P2.54mm_Vertical, symbol Connector:Conn_01x06_Male
- added J39: Delay2_CV, Connector_PinSocket_2.54mm:PinSocket_1x06_P2.54mm_Vertical, symbol Connector:Conn_01x06_Female
- added J6: DelayAudio, Connector_PinSocket_2.54mm:PinSocket_1x06_P2.54mm_Vertical, symbol Connector:Conn_01x06_Female
- added J8: Delay Return, Connector_PinHeader_2.54mm:PinHeader_1x02_P2.54mm_Vertical, symbol Connector:Conn_01x02_Male
Connections:
- net CVInputs/+V is gone; now on net TOP_0V: J1.1 (Pin_1)
- net AudioIO/DELAY1_WET: now also J2.1 (Pin_1)
- net AudioIO/DELAY1_WET_LEVEL: now also J2.2 (Pin_2)
- net AudioIO/DELAY2_SOURCE: now also J2.6 (Pin_6)
- net AudioIO/DELAY2_WET: now also J2.4 (Pin_4)
- net AudioIO/DELAY2_WET_LEVEL: now also J2.3 (Pin_3)
- net AudioIO/INPUT_MIX: now also J2.5 (Pin_5)
- net CVControl/DELAY1_CONTROL: now also J12.2 (Pin_2)
- net CVControl/DELAY1_CV_ATTV: now also J12.3 (Pin_3)
- net CVControl/DELAY1_CV_INPUT: now also J12.5 (Pin_5)
- net CVControl/DELAY1_CV_JOIN_OUT: now also J12.1 (Pin_1)
- net CVControl/DELAY2_CONTROL: now also J39.1 (Pin_1)
- net CVControl/DELAY2_CV_ATTV: now also J39.2 (Pin_2)
- net CVControl/DELAY2_CV_CTRL: now also J39.3 (Pin_3)
- net CVControl/DELAY2_CV_INPUT1: now also J39.4 (Pin_4)
- net CVControl/DELAY2_CV_INPUT2: now also J39.5 (Pin_5)
- net CVInputs/DELAY1_CONTROL: now also J11.2 (Pin_2)
- net CVInputs/DELAY1_CV_ATTV: now also J11.3 (Pin_3)
- net CVInputs/DELAY1_CV_INPUT: now also J11.5 (Pin_5)
- net CVInputs/DELAY2_CONTROL: now also J38.1 (Pin_1)
- net CVInputs/DELAY2_CV_ATTV: now also J38.2 (Pin_2)
- net CVInputs/DELAY2_CV_CTRL: now also J38.3 (Pin_3)
- net CVInputs/DELAY2_CV_INPUT: now also J38.4 (Pin_4)
- net CVInputs/JOIN_CV: now also J38.5 (Pin_5)
- net CVInputs/JOIN_CV_SOURCE: now also J11.1 (Pin_1)
- net DelayOut/DELAY1_WET: now also J6.1 (Pin_1), J8.1 (Pin_1)
- net DelayOut/DELAY2_WET: now also J6.4 (Pin_4), J8.2 (Pin_2)
- net GND: now also H5.1, H6.1
- net InputMix/INPUT_MIX: now also J13.1 (Pin_1), J6.5 (Pin_5)
- net MID_+V: no longer J20.1 (Pin_1)
- net MID_0V: now also J20.1 (Pin_1), H3.1, H4.1, J12.6 (Pin_6), J39.6 (Pin_6)
- net PT2399-Delay-1/AUDIO_IN: now also J32.1 (Pin_1)
- net PT2399-Delay-1/AUDIO_OUT: now also J33.1 (Pin_1)
- net PT2399-Delay-2/AUDIO_IN: now also J32.2 (Pin_2)
- net PT2399-Delay-2/AUDIO_OUT: now also J33.2 (Pin_2)
- net TOP_0V: now also H1.1, H2.1, J11.6 (Pin_6), J38.6 (Pin_6)
- new net: J13.2 (Pin_2), J6.6 (Pin_6)
- new net CVControl/DELAY1_CV_CTRL: J12.4 (Pin_4)
- new net CVInputs/DELAY1_CV_CTRL: J11.4 (Pin_4)
- new net OutputMix/DELAY1_WET_LEVEL: J6.2 (Pin_2)
- new net OutputMix/DELAY2_WET_LEVEL: J6.3 (Pin_3)
Other:
- moved on the sheet: J5

Commit message: Finalising rev 01 of dual digi delay
Connections:
- net GND: now also H1.1, H2.1, H3.1, H4.1
- net MID_0V: no longer H3.1, H4.1
- net TOP_0V: no longer H1.1, H2.1
- net Power/+V renamed +12V
- net Power/-V renamed -12V
Changed lines of the file:
@@
 	12800 9000 12800 7700
 Wire Wire Line
-	12800 7700 11050 7700
+	12800 7700 12500 7700
 Connection ~ 12800 9000
 Wire Wire Line
 	12800 9000 12850 9000
 Wire Wire Line
-	12850 7400 11050 7400
+	12850 7400 12750 7400
 Wire Wire Line
 	11050 7500 11150 7500
@@
 	1    0    0    -1
 $EndComp
-Text Label 10550 2250 3    50   ~ 0
-MID_0V
-Text Label 9800 2250 3    50   ~ 0
-TOP_0V
-Wire Wire Line
-	9800 2250 9800 1950
 Wire Wire Line
 	9800 1600 9750 1600
 Wire Wire Line
 	9750 1950 9800 1950
-Connection ~ 9800 1950
 Wire Wire Line
 	9800 1950 9800 1600
 Wire Wire Line
-	10550 2250 10550 1950
-Wire Wire Line
 	10550 1600 10500 1600
 Wire Wire Line
 	10500 1950 10550 1950
-Connection ~ 10550 1950
 Wire Wire Line
 	10550 1950 10550 1600
 Wire Wire Line
-	11300 2250 11300 1950
+	11300 2250 11300 2150
 Wire Wire Line
 	11300 1600 11250 1600
@@
 Wire Wire Line
 	11300 1950 11300 1600
+Wire Wire Line
+	10550 1950 10550 2150
+Wire Wire Line
+	10550 2150 11300 2150
+Connection ~ 10550 1950
+Connection ~ 11300 2150
+Wire Wire Line
+	11300 2150 11300 1950
+Wire Wire Line
+	9800 1950 9800 2150
+Wire Wire Line
+	9800 2150 10550 2150
+Connection ~ 9800 1950
+Connection ~ 10550 2150
+$Comp
+L power:GND #PWR?
+U 1 1 61822BEE
+P 7700 2550
+F 0 "#PWR?" H 7700 2300 50  0001 C CNN
+F 1 "GND" H 7705 2377 50  0000 C CNN
+F 2 "" H 7700 2550 50  0001 C CNN
+F 3 "" H 7700 2550 50  0001 C CNN
+	1    7700 2550
+	1    0    0    -1
+$EndComp
+$Comp
+L power:+12V #PWR?
+U 1 1 61824BA8
+P 12750 7250
+F 0 "#PWR?" H 12750 7100 50  0001 C CNN
+F 1 "+12V" H 12765 7423 50  0000 C CNN
+F 2 "" H 12750 7250 50  0001 C CNN
+F 3 "" H 12750 7250 50  0001 C CNN
+	1    12750 7250
+	1    0    0    -1
+$EndComp
+$Comp
+L power:-12V #PWR?
+U 1 1 61826230
+P 12500 7250
+F 0 "#PWR?" H 12500 7350 50  0001 C CNN
+F 1 "-12V" H 12515 7423 50  0000 C CNN
+F 2 "" H 12500 7250 50  0001 C CNN
+F 3 "" H 12500 7250 50  0001 C CNN
+	1    12500 7250
+	1    0    0    -1
+$EndComp
+Wire Wire Line
+	12500 7700 12500 7250
+Connection ~ 12500 7700
+Wire Wire Line
+	12500 7700 11050 7700
+Wire Wire Line
+	12750 7400 12750 7250
+Connection ~ 12750 7400
+Wire Wire Line
+	12750 7400 11050 7400
 $EndSCHEMATC

Commit message: Updating digi delay to rev 2
Parts:
- removed J2: DelayAudio, Connector_PinHeader_2.54mm:PinHeader_1x06_P2.54mm_Vertical, symbol Connector:Conn_01x06_Male
- removed J6: DelayAudio, Connector_PinSocket_2.54mm:PinSocket_1x06_P2.54mm_Vertical, symbol Connector:Conn_01x06_Female
- removed NT1: Net-Tie_2, NetTie:NetTie-2_SMD_Pad2.0mm, symbol Device:Net-Tie_2
- added H10, H11, H12, H13, H14, H15, H16, H17, H18, H7, H8, H9: MouseBite, Panelization:mouse-bite-2mm-slot, symbol Panelization:MouseBite
- added H19: Logo_Ammonite-simple, rumblesan-footprints:Logo_Ammonite-simple_10.4mmx12.0mm, symbol Board_Hardware:Logo_Ammonite-simple
- added J17: Delay Audio, Connector_PinSocket_2.54mm:PinSocket_1x04_P2.54mm_Vertical, symbol Connector:Conn_01x04_Female
- added J18: Delay2 Source, Connector_PinSocket_2.54mm:PinSocket_1x03_P2.54mm_Vertical, symbol Connector:Conn_01x03_Female
- added J2: Delay Audio, Connector_PinHeader_2.54mm:PinHeader_1x04_P2.54mm_Vertical, symbol Connector:Conn_01x04_Male
- added J6: Delay2 Source, Connector_PinHeader_2.54mm:PinHeader_1x03_P2.54mm_Vertical, symbol Connector:Conn_01x03_Male
Connections:
- net CVControl/DELAY2_CV_INPUT1 is gone; now on net CVControl/DELAY2_CV_CTRL: J39.4 (Pin_4)
- net CVInputs/-V is gone; now on net GND: J1.4 (Pin_4)
- net MID_+V is gone; now on net +12V: J9.1 (Pin_1)
- net +12V: now also J1.1 (Pin_1), J20.1 (Pin_1)
- net -12V: now also J9.4 (Pin_4)
- net AudioIO/AUDIO_IN: now also J3.3 (Pin_3); no longer J3.1 (Pin_1)
- net AudioIO/DELAY1_WET: now also J2.1 (Pin_1)
- net AudioIO/DELAY1_WET_LEVEL: now also J2.2 (Pin_2)
- net AudioIO/DELAY2_SOURCE: now also J6.2 (Pin_2)
- net AudioIO/DELAY2_WET: now also J2.4 (Pin_4)
- net AudioIO/DELAY2_WET_LEVEL: now also J2.3 (Pin_3)
- net AudioIO/DRY_AUDIO_INPUT: now also J3.2 (Pin_2); no longer J3.3 (Pin_3)
- net AudioIO/FEEDBACK_LEVEL: now also J3.1 (Pin_1); no longer J3.2 (Pin_2)
- net AudioIO/INPUT_MIX: now also J6.3 (Pin_3)
- net CVControl/DELAY2_CONTROL: now also J39.2 (Pin_2); no longer J39.1 (Pin_1)
- net CVControl/DELAY2_CV_ATTV: now also J39.3 (Pin_3); no longer J39.2 (Pin_2)
- net CVControl/DELAY2_CV_CTRL: no longer J39.3 (Pin_3)
- net CVInputs/DELAY2_CONTROL: now also J38.2 (Pin_2); no longer J38.1 (Pin_1)
- net CVInputs/DELAY2_CV_ATTV: now also J38.3 (Pin_3); no longer J38.2 (Pin_2)
- net CVInputs/DELAY2_CV_CTRL: now also J38.4 (Pin_4); no longer J38.3 (Pin_3)
- net CVInputs/DELAY2_CV_INPUT: now also J38.5 (Pin_5); no longer J38.4 (Pin_4)
- net CVInputs/JOIN_CV: now also J38.1 (Pin_1); no longer J38.5 (Pin_5)
- net DelayOut/DELAY1_WET: now also J17.1 (Pin_1), J18.1 (Pin_1)
- net DelayOut/DELAY2_WET: now also J17.4 (Pin_4)
- net GND: now also J1.2 (Pin_2), J1.3 (Pin_3), J11.6 (Pin_6), J12.6 (Pin_6), J16.2 (Pin_2), J20.2 (Pin_2), J20.3 (Pin_3), J20.4 (Pin_4), J3.4 (Pin_4), J31.2 (Pin_2), J38.6 (Pin_6), J39.6 (Pin_6), J7.4 (Pin_4), J9.2 (Pin_2), J9.3 (Pin_3)
- net InputMix/AUDIO_IN: now also J7.3 (Pin_3); no longer J7.1 (Pin_1)
- net InputMix/DELAY_FEEDBACK: now also J7.1 (Pin_1); no longer J7.2 (Pin_2)
- net InputMix/DRY_AUDIO_SOURCE: now also J7.2 (Pin_2); no longer J7.3 (Pin_3)
- net InputMix/INPUT_MIX: now also J18.3 (Pin_3)
- net OutputMix/DELAY1_WET_LEVEL: now also J17.2 (Pin_2)
- net OutputMix/DELAY2_WET_LEVEL: now also J17.3 (Pin_3)
- net at J13.2 (Pin_2): now also J18.2 (Pin_2)
- net CVControl/DELAY2_CV_INPUT2 renamed CVControl/DELAY2_CV_INPUT
- removed net MID_-V: J20.4 (Pin_4), J9.4 (Pin_4)
- removed net MID_0V: J12.6 (Pin_6), J20.1 (Pin_1), J20.2 (Pin_2), J20.3 (Pin_3), J31.2 (Pin_2), J39.6 (Pin_6), J7.4 (Pin_4), J9.2 (Pin_2), J9.3 (Pin_3)
- net PT2399-Delay-1/AUDIO_OUT renamed DelayBuffers/DELAY1_OUT
- net PT2399-Delay-2/AUDIO_OUT renamed DelayBuffers/DELAY2_OUT
- removed net TOP_0V: J1.1 (Pin_1), J1.2 (Pin_2), J1.3 (Pin_3), J11.6 (Pin_6), J16.2 (Pin_2), J3.4 (Pin_4), J38.6 (Pin_6)
- new net AudioIO/DELAY1_WET_TO_2: J6.1 (Pin_1)
- new net CVControl/DELAY2_JOIN_CV_INPUT: J39.1 (Pin_1)
Other:
- moved on the sheet: H1, H2, H3, H4, H5, H6, J1, J10, J12, J13, J16, J20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
