File: dual-digi-delay/audioio.kicad_sch (KiCad schematic)
At the start: 10 parts, among them J1 BananaJack_PanelMount, J2 BananaJack_PanelMount, J4 BananaJack_PanelMount, J5 BananaJack_PanelMount, SW1 SW_SPDT

Commit message: Creating revision 3 of dual digi delay
Other:
- moved on the sheet: DRY_LEVEL1, FEEDBACK1, INPUT_GAIN1, J1, J2, J4, J5, SW1, WET_LEVEL1, WET_LEVEL2
