File: dual-digi-delay/cv-control.kicad_sch (KiCad schematic)
At the start: 55 parts, among them Q1 2N3904, Q2 2N3904, Q3 2N3904, Q4 2N3904, U4 TL074, U5 TL074

Commit message: Creating revision 3 of dual digi delay
Parts:
- C15, C16, C21, C22: value 100nF -> 100nF (X7R)
Connections:
- net +VCC renamed +12V
- net -VCC renamed -12V
Other:
- moved on the sheet: C15, C16, C21, C22, U4E, U5E
