File: dual-digi-delay/cv-inputs.kicad_sch (KiCad schematic)
At the start: 7 parts, among them J3 BananaJack_PanelMount, J6 BananaJack_PanelMount, SW2 SW_SPDT

Commit message: Creating revision 3 of dual digi delay
Connections:
- net +VCC renamed +12V
Changed lines of the file:
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@@
 (kicad_sch (version 20211123) (generator eeschema)
   (paper "A4")
+  (title_block
+    (date "2022-01-13")
+    (rev "v03")
+    (comment 2 "creativecommons.org/licenses/by/4.0/")
+    (comment 3 "License: CC BY 4.0")
+    (comment 4 "Author: Guy John")
+  )
   (no_connect (at 49.53 110.49))
   (wire (pts (xy 45.72 119.38) (xy 45.72 123.19))
@@
     (stroke (width 0) (type default) (color 0 0 0 0))
   )
-  (wire (pts (xy 107.95 88.9) (xy 104.14 88.9))
-    (stroke (width 0) (type default) (color 0 0 0 0))
-  )
   (wire (pts (xy 111.76 129.54) (xy 107.95 129.54))
     (stroke (width 0) (type default) (color 0 0 0 0))
@@
   (wire (pts (xy 104.14 133.35) (xy 104.14 140.97))
     (stroke (width 0) (type default) (color 0 0 0 0))
-  )
-  (wire (pts (xy 104.14 91.44) (xy 107.95 91.44))
-    (stroke (width 0) (type default) (color 0 0 0 0))
-  )
-  (label "GND" (at 43.18 78.74 270)
-    (effects (font (size 1.27 1.27)) (justify right bottom))
-  )
-  (label "+VCC" (at 107.95 88.9 0)
-    (effects (font (size 1.27 1.27)) (justify left bottom))
-  )
-  (label "+VCC" (at 110.49 43.18 90)
-    (effects (font (size 1.27 1.27)) (justify left bottom))
-  )
-  (label "GND" (at 45.72 134.62 270)
-    (effects (font (size 1.27 1.27)) (justify right bottom))
-  )
-  (label "GND" (at 104.14 140.97 270)
-    (effects (font (size 1.27 1.27)) (justify right bottom))
-  )
-  (label "GND" (at 107.95 91.44 0)
-    (effects (font (size 1.27 1.27)) (justify left bottom))
-  )
-  (label "GND" (at 110.49 62.23 270)
-    (effects (font (size 1.27 1.27)) (justify right bottom))
-  )
-  (label "+VCC" (at 104.14 121.92 90)
-    (effects (font (size 1.27 1.27)) (justify left bottom))
   )
   (hierarchical_label "DELAY2_CV_ATTV" (shape input) (at 53.34 127 0)
@@
     (effects (font (size 1.27 1.27)) (justify right))
   )
-  (hierarchical_label "+VCC" (shape input) (at 104.14 88.9 180)
-    (effects (font (size 1.27 1.27)) (justify right))
-  )
   (hierarchical_label "DELAY2_CONTROL" (shape input) (at 111.76 129.54 0)
     (effects (font (size 1.27 1.27)) (justify left))
@@
     (effects (font (size 1.27 1.27)) (justify right))
   )
-  (hierarchical_label "GND" (shape input) (at 104.14 91.44 180)
-    (effects (font (size 1.27 1.27)) (justify right))
-  )
   (hierarchical_label "JOIN_CV_SOURCE" (shape input) (at 45.72 105.41 180)
     (effects (font (size 1.27 1.27)) (justify right))
@@
     (pin "2")
     (pin "3")
+  )
+  (symbol (lib_id "power:GND") (at 110.49 62.23 0) (unit 1)
+    (in_bom yes) (on_board yes)
+    (property "Reference" "#PWR0142" (id 0) (at 110.49 68.58 0)
+      (effects (font (size 1.27 1.27)) hide)
+    )
+    (property "Value" "GND" (id 1) (at 110.617 66.6242 0))
+    (property "Footprint" "" (id 2) (at 110.49 62.23 0)
+      (effects (font (size 1.27 1.27)) hide)
+    )
+    (property "Datasheet" "" (id 3) (at 110.49 62.23 0)
+      (effects (font (size 1.27 1.27)) hide)
+    )
+    (pin "1")
+  )
+  (symbol (lib_id "power:GND") (at 43.18 78.74 0) (unit 1)
+    (in_bom yes) (on_board yes)
+    (property "Reference" "#PWR0141" (id 0) (at 43.18 85.09 0)
+      (effects (font (size 1.27 1.27)) hide)
+    )
+    (property "Value" "GND" (id 1) (at 43.307 83.1342 0))
+    (property "Footprint" "" (id 2) (at 43.18 78.74 0)
+      (effects (font (size 1.27 1.27)) hide)
+    )
+    (property "Datasheet" "" (id 3) (at 43.18 78.74 0)
+      (effects (font (size 1.27 1.27)) hide)
+    )
+    (pin "1")
+  )
+  (symbol (lib_id "power:GND") (at 104.14 140.97 0) (unit 1)
+    (in_bom yes) (on_board yes)
+    (property "Reference" "#PWR0144" (id 0) (at 104.14 147.32 0)
+      (effects (font (size 1.27 1.27)) hide)
+    )
+    (property "Value" "GND" (id 1) (at 104.267 145.3642 0))
+    (property "Footprint" "" (id 2) (at 104.14 140.97 0)
+      (effects (font (size 1.27 1.27)) hide)
+    )
+    (property "Datasheet" "" (id 3) (at 104.14 140.97 0)
+      (effects (font (size 1.27 1.27)) hide)
+    )
+    (pin "1")
+  )
+  (symbol (lib_id "power:+12V") (at 104.14 121.92 0) (unit 1)
+    (in_bom yes) (on_board yes)
+    (property "Reference" "#PWR0145" (id 0) (at 104.14 125.73 0)
+      (effects (font (size 1.27 1.27)) hide)
+    )
+    (property "Value" "+12V" (id 1) (at 104.521 117.5258 0))
+    (property "Footprint" "" (id 2) (at 104.14 121.92 0)
+      (effects (font (size 1.27 1.27)) hide)
+    )
+    (property "Datasheet" "" (id 3) (at 104.14 121.92 0)
+      (effects (font (size 1.27 1.27)) hide)
+    )
+    (pin "1")
   )
   (symbol (lib_id "Switch:SW_SPDT") (at 54.61 107.95 0) (mirror y) (unit 1)
@@
     (pin "3")
   )
+  (symbol (lib_id "power:GND") (at 45.72 134.62 0) (unit 1)
+    (in_bom yes) (on_board yes)
+    (property "Reference" "#PWR0140" (id 0) (at 45.72 140.97 0)
+      (effects (font (size 1.27 1.27)) hide)
+    )
+    (property "Value" "GND" (id 1) (at 45.847 139.0142 0))
+    (property "Footprint" "" (id 2) (at 45.72 134.62 0)
+      (effects (font (size 1.27 1.27)) hide)
+    )
+    (property "Datasheet" "" (id 3) (at 45.72 134.62 0)
+      (effects (font (size 1.27 1.27)) hide)
+    )
+    (pin "1")
+  )
+  (symbol (lib_id "power:+12V") (at 110.49 43.18 0) (unit 1)
+    (in_bom yes) (on_board yes)
+    (property "Reference" "#PWR0143" (id 0) (at 110.49 46.99 0)
+      (effects (font (size 1.27 1.27)) hide)
+    )
+    (property "Value" "+12V" (id 1) (at 110.871 38.7858 0))
+    (property "Footprint" "" (id 2) (at 110.49 43.18 0)
+      (effects (font (size 1.27 1.27)) hide)
+    )
+    (property "Datasheet" "" (id 3) (at 110.49 43.18 0)
+      (effects (font (size 1.27 1.27)) hide)
+    )
+    (pin "1")
+  )
 )
