File: dual-digi-delay/delay-buffers.kicad_sch (KiCad schematic)
At the start: 5 parts, among them U7 TL072

Commit message: Creating revision 3 of dual digi delay
Parts:
- C40, C41: value 100nF -> 100nF (X7R)
Connections:
- net +VCC renamed +12V
- net -VCC renamed -12V
Other:
- moved on the sheet: U7C
Changed lines of the file:
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@@
 (kicad_sch (version 20211123) (generator eeschema)
   (paper "A4")
+  (title_block
+    (date "2022-01-13")
+    (rev "v03")
+    (comment 2 "creativecommons.org/licenses/by/4.0/")
+    (comment 3 "License: CC BY 4.0")
+    (comment 4 "Author: Guy John")
+  )
   (junction (at 233.68 63.5) (diameter 0) (color 0 0 0 0)
   )
@@
     (stroke (width 0) (type default) (color 0 0 0 0))
   )
-  (wire (pts (xy 223.52 104.14) (xy 227.33 104.14))
-    (stroke (width 0) (type default) (color 0 0 0 0))
-  )
   (wire (pts (xy 170.18 71.12) (xy 172.72 71.12))
     (stroke (width 0) (type default) (color 0 0 0 0))
   )
+  (wire (pts (xy 252.73 63.5) (xy 252.73 68.58))
+    (stroke (width 0) (type default) (color 0 0 0 0))
+  )
+  (wire (pts (xy 227.33 88.9) (xy 233.68 88.9))
+    (stroke (width 0) (type default) (color 0 0 0 0))
+  )
   (wire (pts (xy 144.78 96.52) (xy 154.94 96.52))
     (stroke (width 0) (type default) (color 0 0 0 0))
@@
     (stroke (width 0) (type default) (color 0 0 0 0))
   )
-  (wire (pts (xy 227.33 106.68) (xy 223.52 106.68))
-    (stroke (width 0) (type default) (color 0 0 0 0))
-  )
   (wire (pts (xy 144.78 68.58) (xy 154.94 68.58))
     (stroke (width 0) (type default) (color 0 0 0 0))
@@
     (stroke (width 0) (type default) (color 0 0 0 0))
   )
+  (wire (pts (xy 227.33 63.5) (xy 233.68 63.5))
+    (stroke (width 0) (type default) (color 0 0 0 0))
+  )
   (wire (pts (xy 152.4 73.66) (xy 152.4 78.74))
     (stroke (width 0) (type default) (color 0 0 0 0))
@@
     (stroke (width 0) (type default) (color 0 0 0 0))
   )
+  (wire (pts (xy 227.33 88.9) (xy 227.33 91.44))
+    (stroke (width 0) (type default) (color 0 0 0 0))
+  )
   (wire (pts (xy 233.68 63.5) (xy 233.68 66.04))
     (stroke (width 0) (type default) (color 0 0 0 0))
   )
-  (wire (pts (xy 247.65 83.82) (xy 247.65 88.9))
-    (stroke (width 0) (type default) (color 0 0 0 0))
-  )
-  (wire (pts (xy 222.25 63.5) (xy 233.68 63.5))
+  (wire (pts (xy 252.73 88.9) (xy 252.73 83.82))
     (stroke (width 0) (type default) (color 0 0 0 0))
   )
@@
     (stroke (width 0) (type default) (color 0 0 0 0))
   )
-  (wire (pts (xy 247.65 63.5) (xy 247.65 68.58))
-    (stroke (width 0) (type default) (color 0 0 0 0))
-  )
   (wire (pts (xy 172.72 106.68) (xy 172.72 99.06))
     (stroke (width 0) (type default) (color 0 0 0 0))
@@
     (stroke (width 0) (type default) (color 0 0 0 0))
   )
-  (wire (pts (xy 222.25 88.9) (xy 233.68 88.9))
-    (stroke (width 0) (type default) (color 0 0 0 0))
-  )
   (wire (pts (xy 144.78 100.33) (xy 144.78 96.52))
     (stroke (width 0) (type default) (color 0 0 0 0))
@@
     (stroke (width 0) (type default) (color 0 0 0 0))
   )
-  (wire (pts (xy 223.52 101.6) (xy 227.33 101.6))
-    (stroke (width 0) (type default) (color 0 0 0 0))
-  )
-  (wire (pts (xy 233.68 76.2) (xy 222.25 76.2))
+  (wire (pts (xy 233.68 76.2) (xy 227.33 76.2))
     (stroke (width 0) (type default) (color 0 0 0 0))
   )
@@
     (stroke (width 0) (type default) (color 0 0 0 0))
   )
-  (wire (pts (xy 233.68 63.5) (xy 247.65 63.5))
+  (wire (pts (xy 227.33 76.2) (xy 227.33 78.74))
+    (stroke (width 0) (type default) (color 0 0 0 0))
+  )
+  (wire (pts (xy 233.68 63.5) (xy 252.73 63.5))
     (stroke (width 0) (type default) (color 0 0 0 0))
   )
@@
     (stroke (width 0) (type default) (color 0 0 0 0))
   )
-  (wire (pts (xy 233.68 88.9) (xy 247.65 88.9))
+  (wire (pts (xy 233.68 88.9) (xy 252.73 88.9))
     (stroke (width 0) (type default) (color 0 0 0 0))
   )
@@
     (stroke (width 0) (type default) (color 0 0 0 0))
   )
+  (wire (pts (xy 227.33 60.96) (xy 227.33 63.5))
+    (stroke (width 0) (type default) (color 0 0 0 0))
+  )
   (wire (pts (xy 172.72 78.74) (xy 172.72 71.12))
     (stroke (width 0) (type default) (color 0 0 0 0))
-  )
-  (label "GND" (at 223.52 104.14 180)
-    (effects (font (size 1.27 1.27)) (justify right bottom))
-  )
-  (label "+VCC" (at 223.52 101.6 180)
-    (effects (font (size 1.27 1.27)) (justify right bottom))
-  )
-  (label "-VCC" (at 223.52 106.68 180)
-    (effects (font (size 1.27 1.27)) (justify right bottom))
-  )
-  (label "GND" (at 144.78 110.49 270)
-    (effects (font (size 1.27 1.27)) (justify right bottom))
-  )
-  (label "-VCC" (at 222.25 88.9 180)
-    (effects (font (size 1.27 1.27)) (justify right bottom))
-  )
-  (label "GND" (at 222.25 76.2 180)
-    (effects (font (size 1.27 1.27)) (justify right bottom))
-  )
-  (label "GND" (at 144.78 82.55 270)
-    (effects (font (size 1.27 1.27)) (justify right bottom))
-  )
-  (label "+VCC" (at 222.25 63.5 180)
-    (effects (font (size 1.27 1.27)) (justify right bottom))
   )
   (hierarchical_label "DELAY1_IN" (shape input) (at 139.7 68.58 180)
@@
   (hierarchical_label "DELAY2_IN" (shape input) (at 139.7 96.52 180)
     (effects (font (size 1.27 1.27)) (justify right))
-  )
-  (hierarchical_label "+VCC" (shape input) (at 227.33 101.6 0)
-    (effects (font (size 1.27 1.27)) (justify left))
-  )
-  (hierarchical_label "-VCC" (shape input) (at 227.33 106.68 0)
-    (effects (font (size 1.27 1.27)) (justify left))
-  )
-  (hierarchical_label "GND" (shape input) (at 227.33 104.14 0)
-    (effects (font (size 1.27 1.27)) (justify left))
   )
   (hierarchical_label "DELAY1_OUT" (shape input) (at 175.26 71.12 0)
@@
     (pin "7")
   )
-  (symbol (lib_id "Amplifier_Operational:TL072") (at 250.19 76.2 0) (unit 3)
-    (in_bom yes) (on_board yes)
-    (property "Reference" "U7" (id 0) (at 249.1232 75.0316 0)
-      (effects (font (size 1.27 1.27)) (justify left))
-    )
-    (property "Value" "TL072" (id 1) (at 249.1232 77.343 0)
-      (effects (font (size 1.27 1.27)) (justify left))
-    )
-    (property "Footprint" "Rumblesan_Footprints:DIP-8_W7.62mm_Socket" (id 2) (at 250.19 76.2 0)
-      (effects (font (size 1.27 1.27)) hide)
-    )
-    (property "Datasheet" "http://www.ti.com/lit/ds/symlink/tl071.pdf" (id 3) (at 250.19 76.2 0)
+  (symbol (lib_id "Amplifier_Operational:TL072") (at 255.27 76.2 0) (unit 3)
+    (in_bom yes) (on_board yes)
+    (property "Reference" "U7" (id 0) (at 254.2032 75.0316 0)
+      (effects (font (size 1.27 1.27)) (justify left))
+    )
+    (property "Value" "TL072" (id 1) (at 254.2032 77.343 0)
+      (effects (font (size 1.27 1.27)) (justify left))
+    )
+    (property "Footprint" "Rumblesan_Footprints:DIP-8_W7.62mm_Socket" (id 2) (at 255.27 76.2 0)
+      (effects (font (size 1.27 1.27)) hide)
+    )
+    (property "Datasheet" "http://www.ti.com/lit/ds/symlink/tl071.pdf" (id 3) (at 255.27 76.2 0)
       (effects (font (size 1.27 1.27)) hide)
     )
@@
       (effects (font (size 1.27 1.27)) (justify right))
     )
-    (property "Value" "100nF" (id 1) (at 236.601 70.993 0)
+    (property "Value" "100nF (X7R)" (id 1) (at 236.601 70.993 0)
       (effects (font (size 1.27 1.27)) (justify right))
     )
@@
       (effects (font (size 1.27 1.27)) (justify right))
     )
-    (property "Value" "100nF" (id 1) (at 236.601 83.693 0)
+    (property "Value" "100nF (X7R)" (id 1) (at 236.601 83.693 0)
       (effects (font (size 1.27 1.27)) (justify right))
     )
@@
     (pin "2")
   )
+  (symbol (lib_id "power:GND") (at 144.78 110.49 0) (unit 1)
+    (in_bom yes) (on_board yes)
+    (property "Reference" "#PWR0150" (id 0) (at 144.78 116.84 0)
+      (effects (font (size 1.27 1.27)) hide)
+    )
+    (property "Value" "GND" (id 1) (at 144.907 114.8842 0))
+    (property "Footprint" "" (id 2) (at 144.78 110.49 0)
+      (effects (font (size 1.27 1.27)) hide)
+    )
+    (property "Datasheet" "" (id 3) (at 144.78 110.49 0)
+      (effects (font (size 1.27 1.27)) hide)
+    )
+    (pin "1")
+  )
+  (symbol (lib_id "power:-12V") (at 227.33 91.44 180) (unit 1)
+    (in_bom yes) (on_board yes)
+    (property "Reference" "#PWR0146" (id 0) (at 227.33 93.98 0)
+      (effects (font (size 1.27 1.27)) hide)
+    )
+    (property "Value" "-12V" (id 1) (at 226.949 95.8342 0))
+    (property "Footprint" "" (id 2) (at 227.33 91.44 0)
+      (effects (font (size 1.27 1.27)) hide)
+    )
+    (property "Datasheet" "" (id 3) (at 227.33 91.44 0)
+      (effects (font (size 1.27 1.27)) hide)
+    )
+    (pin "1")
+  )
+  (symbol (lib_id "power:+12V") (at 227.33 60.96 0) (unit 1)
+    (in_bom yes) (on_board yes)
+    (property "Reference" "#PWR0148" (id 0) (at 227.33 64.77 0)
+      (effects (font (size 1.27 1.27)) hide)
+    )
+    (property "Value" "+12V" (id 1) (at 227.711 56.5658 0))
+    (property "Footprint" "" (id 2) (at 227.33 60.96 0)
+      (effects (font (size 1.27 1.27)) hide)
+    )
+    (property "Datasheet" "" (id 3) (at 227.33 60.96 0)
+      (effects (font (size 1.27 1.27)) hide)
+    )
+    (pin "1")
+  )
+  (symbol (lib_id "power:GND") (at 227.33 78.74 0) (unit 1)
+    (in_bom yes) (on_board yes)
+    (property "Reference" "#PWR0147" (id 0) (at 227.33 85.09 0)
+      (effects (font (size 1.27 1.27)) hide)
+    )
+    (property "Value" "GND" (id 1) (at 227.457 83.1342 0))
+    (property "Footprint" "" (id 2) (at 227.33 78.74 0)
+      (effects (font (size 1.27 1.27)) hide)
+    )
+    (property "Datasheet" "" (id 3) (at 227.33 78.74 0)
+      (effects (font (size 1.27 1.27)) hide)
+    )
+    (pin "1")
+  )
+  (symbol (lib_id "power:GND") (at 144.78 82.55 0) (unit 1)
+    (in_bom yes) (on_board yes)
+    (property "Reference" "#PWR0149" (id 0) (at 144.78 88.9 0)
+      (effects (font (size 1.27 1.27)) hide)
+    )
+    (property "Value" "GND" (id 1) (at 144.907 86.9442 0))
+    (property "Footprint" "" (id 2) (at 144.78 82.55 0)
+      (effects (font (size 1.27 1.27)) hide)
+    )
+    (property "Datasheet" "" (id 3) (at 144.78 82.55 0)
+      (effects (font (size 1.27 1.27)) hide)
+    )
+    (pin "1")
+  )
 )
