File: dual-digi-delay/delay-out.kicad_sch (KiCad schematic)
At the start: 11 parts, among them U2 TL072

Commit message: Creating revision 3 of dual digi delay
Parts:
- C1, C6: value 100nF -> 100nF (X7R)
Connections:
- net +VCC renamed +12V
- net -VCC renamed -12V
Other:
- moved on the sheet: C1, C6, U2C
