File: dual-digi-delay/dual-digi-delay.kicad_sch (KiCad schematic)
At the start: 46 parts, among them J10 Delay Audio, J11 Delay2 Source, J12 Input Audio, J13 Delay1_CV, J14 Delay2_CV, J15 MidBoardPowerSend, J16 Delay Send, J17 Delay Return, J18 Delay Time Control, J19 LowerBoardPowerSend, J20 Main Power, J21 Delay Return, J22 Delay Send, J23 Delay Time Control, J24 MidBoardPowerRecv, J25 Delay Out, J26 Delay Audio, J27 Delay2_CV, J28 Output Audio, J29 Delay2 Source, J30 TopBoardPowerRecv, J31 Feedback Audio, J32 Input Audio, J33 Delay1_CV, J7 Output Audio, J8 Delay Out, J9 Feedback Audio

Commit message: Creating revision 3 of dual digi delay
Connections:
- net +12V: no longer J20.1 (Pin_1)
- net -12V: no longer J20.4 (Pin_4)
- new net Power/+VCC: J20.1 (Pin_1)
- new net Power/-VCC: J20.4 (Pin_4)
Other:
- sheet AudioIO ports: added none; removed GND
- sheet CVControl ports: added none; removed +VCC, -VCC, GND
- sheet CVInputs ports: added none; removed +VCC, GND
- sheet DelayBuffers ports: added none; removed +VCC, -VCC, GND
- sheet DelayOut ports: added none; removed +VCC, -VCC, GND
- sheet InputMix ports: added none; removed +VCC, -VCC, GND
- sheet OutputMix ports: added none; removed +VCC, -VCC, GND
- sheet PT2399-Delay-1 ports: added none; removed +VCC, GND
- sheet PT2399-Delay-2 ports: added none; removed +VCC, GND
- sheet Power ports: added none; removed +5V, GND
- moved on the sheet: J19, J20, J24, J30
