File: dual-digi-delay/inputmix.kicad_sch (KiCad schematic)
At the start: 14 parts, among them U3 TL072

Commit message: Creating revision 3 of dual digi delay
Parts:
- C10, C12: value 100nF -> 100nF (X7R)
Connections:
- net 0V is gone; now on net GND: U3.5 (+)
- net +VCC renamed +12V
- net -VCC renamed -12V
Other:
- moved on the sheet: C10, C12, U3C
