File: dual-digi-delay/outputmix.kicad_sch (KiCad schematic)
At the start: 16 parts, among them U1 TL072

Commit message: Creating revision 3 of dual digi delay
Parts:
- C4, C5: value 100nF -> 100nF (X7R)
Connections:
- net +VCC renamed +12V
- net -VCC renamed -12V
Other:
- moved on the sheet: C4, C5, U1C
