File: dual-digi-delay/power.kicad_sch (KiCad schematic)
At the start: 7 parts, among them U9 LM7805_TO220

Commit message: Creating revision 3 of dual digi delay
Parts:
- C56, C59: value 100nF -> 100nF (X7R)
Connections:
- net +VCC: now also D15.2 (A); no longer C59.2, C60.1, D15.1 (K), U9.1 (VI)
- net -VCC: no longer C58.2
- net GND: no longer D15.2 (A), D16.1 (K)
- new net +12V: C59.2, C60.1, D15.1 (K), U9.1 (VI)
- new net -12V: C58.2, D16.1 (K)
Other:
- moved on the sheet: D15, D16
