File: blank-panels/4u-2col-spiral-tiled/4u-2col-spiral-tiled.kicad_pcb (KiCad board)
At the start: 2 copper layers, 50.5 x 175 mm, 5 parts

Commit message: Tweaking blank panel projects
Other:
- net class Default removed
