File: chaos-suite/4u-simple-integrator/4u-simple-integrator.kicad_pcb (KiCad board)
At the start: 2 copper layers, 0 parts

Commit message: Final tweaks to simple integrator
Parts:
- added C1: 1nF (poly), Rumblesan_Footprints:C_Rect_L7.0mm_W3.5mm_P5.00mm, F.Cu at (105.4, 84.3)
- added C2: 1nF (poly), Rumblesan_Footprints:C_Rect_L7.0mm_W3.5mm_P5.00mm, F.Cu at (105.4, 108.5)
- added C3: 100nF (X7R), Rumblesan_Footprints:C_Rect_L7.0mm_W3.5mm_P5.00mm, F.Cu at (112.5, 103.5)
- added C4: 100nF (X7R), Rumblesan_Footprints:C_Rect_L7.0mm_W3.5mm_P5.00mm, F.Cu at (112.5, 84.3)
- added C7: 1uF, Capacitor_THT:CP_Radial_D5.0mm_P2.00mm, F.Cu at (108.3, 52.5)
- added C8: 1uF, Capacitor_THT:CP_Radial_D5.0mm_P2.00mm, F.Cu at (114.7, 52.5)
- added D1: 1N5818, Rumblesan_Footprints:D_DO-41_SOD81_P10.16mm_Horizontal, F.Cu at (104.5, 52.5)
- added D2: 1N5818, Rumblesan_Footprints:D_DO-41_SOD81_P10.16mm_Horizontal, F.Cu at (120.7, 42.3)
- added H1: MountingHole_Pad, MountingHole:MountingHole_3.2mm_M3_Pad, F.Cu at (120.9, 177.3)
- added H2: MountingHole_Pad, MountingHole:MountingHole_3.2mm_M3_Pad, F.Cu at (104.1, 34.8)
- added H3: MountingHole_Pad, MountingHole:MountingHole_3.2mm_M3_Pad, F.Cu at (94.2, 177.3)
- added H4: MountingHole_Pad, MountingHole:MountingHole_3.2mm_M3_Pad, F.Cu at (77.5, 34.8)
- added H5: MouseBite, Panelization:mouse-bite-2.54mm-slot, F.Cu at (99.2, 77.9)
- added H6: MouseBite, Panelization:mouse-bite-2.54mm-slot, F.Cu at (99.2, 135.0)
- added H7: MouseBite, Panelization:mouse-bite-2.54mm-slot, F.Cu at (99.2, 163.7)
- added H8: MouseBite, Panelization:mouse-bite-2.54mm-slot, F.Cu at (99.2, 48.6)
- added H9: MouseBite, Panelization:mouse-bite-2.54mm-slot, F.Cu at (99.2, 106.4)
- added J1: BananaJack_PanelMount, Rumblesan_Footprints:BananaJack_THT_JohnsonCinch_108-09, B.Cu at (85.9, 96.5)
- added J10: I2_Main, Connector_PinHeader_2.54mm:PinHeader_1x04_P2.54mm_Vertical, B.Cu at (109.0, 144.0)
- added J11: 4U_Power, Rumblesan_Footprints:4u_Power_Molex_KK-254_P2.54mm, B.Cu at (113.0, 35.6)
- added J2: BananaJack_PanelMount, Rumblesan_Footprints:BananaJack_THT_JohnsonCinch_108-09, B.Cu at (85.9, 172.7)
- added J3: BananaJack_PanelMount, Rumblesan_Footprints:BananaJack_THT_JohnsonCinch_108-09, B.Cu at (85.9, 58.4)
- added J4: BananaJack_PanelMount, Rumblesan_Footprints:BananaJack_THT_JohnsonCinch_108-09, B.Cu at (85.9, 39.4)
- added J5: BananaJack_PanelMount, Rumblesan_Footprints:BananaJack_THT_JohnsonCinch_108-09, B.Cu at (85.9, 134.6)
- added J6: BananaJack_PanelMount, Rumblesan_Footprints:BananaJack_THT_JohnsonCinch_108-09, B.Cu at (85.9, 115.6)
- added J7: I1_Ctrl, Connector_PinSocket_2.54mm:PinSocket_1x04_P2.54mm_Vertical, F.Cu at (90.2, 68.1)
- added J8: I2_Ctrl, Connector_PinSocket_2.54mm:PinSocket_1x04_P2.54mm_Vertical, F.Cu at (82.3, 144.0)
- added J9: I1_Main, Connector_PinHeader_2.54mm:PinHeader_1x04_P2.54mm_Vertical, B.Cu at (116.8, 68.1)
- added R1: 100k, Rumblesan_Footprints:Resistor_THT_L6.3mm_D2.5mm_P10.16mm_Horizontal, F.Cu at (105.4, 70.7)
- added R2: 100k, Rumblesan_Footprints:Resistor_THT_L6.3mm_D2.5mm_P10.16mm_Horizontal, F.Cu at (109.0, 126.4)
- added R3: 100k, Rumblesan_Footprints:Resistor_THT_L6.3mm_D2.5mm_P10.16mm_Horizontal, F.Cu at (109.0, 79.4)
- added R4: 100k, Rumblesan_Footprints:Resistor_THT_L6.3mm_D2.5mm_P10.16mm_Horizontal, F.Cu at (109.0, 113.4)
- added R5: 10k, Rumblesan_Footprints:Resistor_THT_L6.3mm_D2.5mm_P10.16mm_Horizontal, F.Cu at (117.1, 79.4)
- added R6: 10k, Rumblesan_Footprints:Resistor_THT_L6.3mm_D2.5mm_P10.16mm_Horizontal, F.Cu at (117.1, 113.4)
- added R7: 10k, Rumblesan_Footprints:Resistor_THT_L6.3mm_D2.5mm_P10.16mm_Horizontal, F.Cu at (120.1, 89.5)
- added R8: 10k, Rumblesan_Footprints:Resistor_THT_L6.3mm_D2.5mm_P10.16mm_Horizontal, F.Cu at (120.1, 103.3)
- added RV1: 100k, Rumblesan_Footprints:Potentiometer_Alpha_RD901F-40-00D_Single_Vertical_CircularHoles, B.Cu at (85.9, 77.5)
- added RV2: 100k, Rumblesan_Footprints:Potentiometer_Alpha_RD901F-40-00D_Single_Vertical_CircularHoles, B.Cu at (85.9, 153.7)
- added U1: TL074, Rumblesan_Footprints:DIP-14_W7.62mm_Socket, F.Cu at (104.9, 100.2)
Routing:
- net +12V: track 0.00 -> 64.1 mm
- net -12V: track 0.00 -> 63.7 mm
- net Net-(J10-Pad1): track 0.00 -> 59.2 mm
- net Net-(C2-Pad2): track 0.00 -> 53.5 mm
- net Net-(J4-Pad1): track 0.00 -> 38.4 mm
- net Net-(C1-Pad2): track 0.00 -> 34.7 mm
- net Net-(J6-Pad1): track 0.00 -> 32.7 mm
- net Net-(R7-Pad2): track 0.00 -> 27.0 mm
- net Net-(J10-Pad2): track 0.00 -> 18.7 mm
- net Net-(J8-Pad2): track 0.00 -> 18.4 mm
- net Net-(R2-Pad2): track 0.00 -> 18.3 mm
- net Net-(RV1-Pad2): track 0.00 -> 18.3 mm
- net Net-(J2-Pad1): track 0.00 -> 16.9 mm
- net Net-(RV1-Pad3): track 0.00 -> 16.9 mm
- net Net-(C1-Pad1): track 0.00 -> 16.7 mm
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- added copper zone on B.Cu, net GND
- added copper zone on F.Cu, net GND
Other:
- board outline added: 50.8 x 149.9 mm
- net class Default removed
- net class Power removed
- net class Signal removed
- board text added: "Simple Integrator r01"

Commit message: finalising rev01 of simple integrator
Parts:
- J11: moved to F.Cu

Commit message: Updating simple integrator to rev2
Parts:
- removed C7, C8: 1uF, Capacitor_THT:CP_Radial_D5.0mm_P2.00mm
- removed H5, H6, H7, H8, H9: MouseBite, Panelization:mouse-bite-2.54mm-slot
- added C5: 10uF, rumblesan-standard-parts:CP_Radial_D5.0mm_P2.00mm, F.Cu at (126.4, 47.0)
- added C6: 10uF, rumblesan-standard-parts:CP_Radial_D5.0mm_P2.00mm, F.Cu at (133.3, 47.0)
- added R10: 330r, rumblesan-standard-parts:R_Axial_DIN0207_L6.3mm_D2.5mm_P10.16mm_Horizontal, F.Cu at (123.2, 90.8)
- added R11: 10k, rumblesan-standard-parts:R_Axial_DIN0207_L6.3mm_D2.5mm_P10.16mm_Horizontal, F.Cu at (126.2, 125.1)
- added R12: 10k, rumblesan-standard-parts:R_Axial_DIN0207_L6.3mm_D2.5mm_P10.16mm_Horizontal, F.Cu at (126.2, 90.8)
- added R9: 330r, rumblesan-standard-parts:R_Axial_DIN0207_L6.3mm_D2.5mm_P10.16mm_Horizontal, F.Cu at (123.2, 125.1)
- added mouse-bite-2.54mm-slot: VAL**, Panelization:mouse-bite-2.54mm-slot, F.Cu at (118.1, 165.1)
- added mouse-bite-2.54mm-slot: VAL**, Panelization:mouse-bite-2.54mm-slot, F.Cu at (118.1, 146.1)
- added mouse-bite-2.54mm-slot: VAL**, Panelization:mouse-bite-2.54mm-slot, F.Cu at (118.1, 50.8)
- added mouse-bite-2.54mm-slot: VAL**, Panelization:mouse-bite-2.54mm-slot, F.Cu at (118.1, 127.0)
- added mouse-bite-2.54mm-slot: VAL**, Panelization:mouse-bite-2.54mm-slot, F.Cu at (118.1, 69.8)
- added mouse-bite-2.54mm-slot: VAL**, Panelization:mouse-bite-2.54mm-slot, F.Cu at (118.1, 108.0)
- added mouse-bite-2.54mm-slot: VAL**, Panelization:mouse-bite-2.54mm-slot, F.Cu at (118.1, 88.9)
- C1, C2: value 1nF (poly) -> 1nF; footprint Rumblesan_Footprints:C_Rect_L7.0mm_W3.5mm_P5.00mm -> rumblesan-standard-parts:C_Rect_L7.0mm_W3.5mm_P5.00mm
- C3, C4: value 100nF (X7R) -> 100nF; footprint Rumblesan_Footprints:C_Rect_L7.0mm_W3.5mm_P5.00mm -> rumblesan-standard-parts:C_Rect_L7.0mm_W3.5mm_P5.00mm
- D1, D2: footprint Rumblesan_Footprints:D_DO-41_SOD81_P10.16mm_Horizontal -> rumblesan-standard-parts:D_DO-41_SOD81_P10.16mm_Horizontal
- J1, J2, J3, J4, J5, J6: footprint Rumblesan_Footprints:BananaJack_THT_JohnsonCinch_108-09 -> rumblesan-standard-parts:BananaJack_THT_JohnsonCinch_108-09
- J10: value I2_Main -> I1_Main
- J11: footprint Rumblesan_Footprints:4u_Power_Molex_KK-254_P2.54mm -> 4u-power:4u_Power_Molex_KK-254_P2.54mm
- J7: value I1_Ctrl -> I2_Ctrl
- J8: value I2_Ctrl -> I1_Ctrl
- J9: value I1_Main -> I2_Main
- R1, R2, R7, R8: footprint Rumblesan_Footprints:Resistor_THT_L6.3mm_D2.5mm_P10.16mm_Horizontal -> rumblesan-standard-parts:R_Axial_DIN0207_L6.3mm_D2.5mm_P10.16mm_Horizontal
- R3, R4: value 100k -> 330r; footprint Rumblesan_Footprints:Resistor_THT_L6.3mm_D2.5mm_P10.16mm_Horizontal -> rumblesan-standard-parts:R_Axial_DIN0207_L6.3mm_D2.5mm_P10.16mm_Horizontal
- R5, R6: value 10k -> 100k (optional); footprint Rumblesan_Footprints:Resistor_THT_L6.3mm_D2.5mm_P10.16mm_Horizontal -> rumblesan-standard-parts:R_Axial_DIN0207_L6.3mm_D2.5mm_P10.16mm_Horizontal
- RV1, RV2: footprint Rumblesan_Footprints:Potentiometer_Alpha_RD901F-40-00D_Single_Vertical_CircularHoles -> rumblesan-standard-parts:Potentiometer_Alpha_RD901F-40-00D_Single_Vertical
- U1: footprint Rumblesan_Footprints:DIP-14_W7.62mm_Socket -> rumblesan-standard-parts:DIP-14_W7.62mm_Socket
- moved R5 51.8 mm to (139.1, 126.2), turned to 180 degrees
- moved C1 43.2 mm to (135.9, 114.9)
- moved C4 40.1 mm to (130.8, 119.9), turned to 90 degrees
- moved R1 35.9 mm to (139.1, 83.2), turned to 180 degrees
- moved H4 35.6 mm to (113.0, 35.6)
- moved R7 34.8 mm to (128.9, 123.2), turned to 0 degrees
- moved H2 34.3 mm to (138.4, 35.6)
- moved U1 33.8 mm to (138.4, 104.2), turned to -90 degrees
- moved R6 32.6 mm to (139.1, 89.3), turned to 180 degrees
- moved C2 31.4 mm to (135.9, 101.0)
- moved R2 30.7 mm to (139.1, 132.3), turned to 180 degrees
- moved R4 25.5 mm to (128.9, 129.3), turned to 0 degrees
- moved R3 21.1 mm to (128.9, 86.2), turned to 0 degrees
- moved J1 19.7 mm to (105.4, 98.4), turned to 180 degrees
- moved J2 19.7 mm to (105.4, 174.6), turned to 180 degrees
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Connections:
- C2 pad 1: Net-(R2-Pad2) -> Net-(C2-Pad1)
- J10 pad 3: Net-(C2-Pad2) -> GND
- J10 pad 4: GND -> Net-(J10-Pad4)
- J7 pad 2: Net-(J4-Pad1) -> Net-(J7-Pad2)
- J7 pad 3: GND -> Net-(J4-Pad1)
- J7 pad 4: Net-(RV1-Pad2) -> GND
- J8 pad 2: Net-(J8-Pad2) -> Net-(J6-Pad1)
- J8 pad 3: Net-(J6-Pad1) -> GND
- J8 pad 4: GND -> Net-(J8-Pad4)
- J9 pad 1: Net-(R7-Pad2) -> Net-(J9-Pad1)
- J9 pad 2: Net-(C1-Pad2) -> Net-(J9-Pad2)
- J9 pad 3: GND -> Net-(J9-Pad3)
- J9 pad 4: Net-(R1-Pad1) -> GND
- R1 pad 1: Net-(R1-Pad1) -> Net-(C2-Pad1)
- R1 pad 2: Net-(C1-Pad1) -> Net-(J9-Pad2)
- R2 pad 1: Net-(J10-Pad2) -> Net-(C1-Pad1)
- R2 pad 2: Net-(R2-Pad2) -> Net-(J10-Pad4)
- R3 pad 1: Net-(C1-Pad1) -> Net-(J9-Pad3)
- R3 pad 2: Net-(C1-Pad2) -> Net-(C2-Pad2)
- R4 pad 1: Net-(R2-Pad2) -> Net-(J10-Pad2)
- R4 pad 2: Net-(C2-Pad2) -> Net-(C1-Pad2)
- R5 pad 2: Net-(R5-Pad2) -> Net-(C1-Pad1)
- R6 pad 2: Net-(R6-Pad2) -> Net-(C2-Pad1)
- R7 pad 1: Net-(R5-Pad2) -> Net-(R11-Pad2)
- R7 pad 2: Net-(R7-Pad2) -> Net-(C1-Pad2)
- R8 pad 1: Net-(R6-Pad2) -> Net-(R12-Pad2)
- R8 pad 2: Net-(J10-Pad1) -> Net-(C2-Pad2)
- RV1 pad 2: Net-(RV1-Pad2) -> Net-(J7-Pad2)
- RV2 pad 2: Net-(J8-Pad2) -> Net-(J8-Pad4)
- U1 pad 2: Net-(R2-Pad2) -> Net-(C2-Pad1)
- U1 pad 6: Net-(R6-Pad2) -> Net-(R12-Pad2)
- U1 pad 7: Net-(J10-Pad1) -> Net-(R10-Pad2)
- U1 pad 8: Net-(R7-Pad2) -> Net-(R11-Pad1)
- U1 pad 9: Net-(R5-Pad2) -> Net-(R11-Pad2)
Routing:
- net Net-(J10-Pad1): track 59.2 -> 14.5 mm
- net Net-(C2-Pad2): track 53.5 -> 20.3 mm
- net Net-(C2-Pad1): track 0.00 -> 28.8 mm
- net Net-(R7-Pad2): track 27.0 -> 0.00 mm
- net Net-(J9-Pad1): track 0.00 -> 22.5 mm
- net Net-(J8-Pad4): track 0.00 -> 21.3 mm
- net Net-(J7-Pad2): track 0.00 -> 18.6 mm
- net Net-(J8-Pad2): track 18.4 -> 0.00 mm
- net Net-(R2-Pad2): track 18.3 -> 0.00 mm
- net Net-(RV1-Pad2): track 18.3 -> 0.00 mm
- net Net-(J9-Pad3): track 0.00 -> 17.7 mm
- net Net-(J10-Pad4): track 0.00 -> 17.2 mm
- net Net-(C1-Pad2): track 34.7 -> 19.9 mm
- net Net-(R10-Pad2): track 0.00 -> 14.6 mm
- net Net-(R11-Pad1): track 0.00 -> 14.6 mm
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Other:
- board size 50.8 x 149.9 mm -> 48.3 x 152.4 mm
- board text added: "Simple Integrator r02"
- board text removed: "Simple Integrator r01"
