File: banana-bread-board-helper/banana-bread-board-helper.kicad_pcb (KiCad board)
At the start: 2 copper layers, 31 x 21 mm, 3 parts, among them J1 BananaJack_PCBMount, J2 BananaJack_PCBMount, J3 Conn_02x04_Odd_Even

Commit message: Updating banana bread board helper
Parts:
- J1, J2: footprint rumblesan-footprints:Deltron_571_PCB_BananaJack -> rumblesan-standard-parts:Deltron_571_PCB_BananaJack
Other:
- net class Default removed
- net class Power removed
- net class Signal removed
